File: EXTENSIONS/Analog/2022.USB French Bar 2/USB French Bar 2.brd (EAGLE design)
At the start: 51 x 50 mm, 11 parts, among them X1 USB-A

Commit message: 2022 Authoring Lights
Parts:
- moved JP1 4.00 mm to (43.0, 28.0)
- moved JP3 4.00 mm to (43.0, 22.0)
- moved RN1 0.50 mm to (25.0, 11.5)
Routing:
- net N$1: track 79.9 -> 0.00 mm
- net VCC: track 45.7 -> 0.00 mm
- net N$3: track 40.1 -> 0.00 mm
- net N$4: track 39.6 -> 0.00 mm
- net N$8: track 23.8 -> 0.00 mm
- net N$2: track 21.9 -> 0.00 mm
- net N$5: track 13.7 -> 0.00 mm
- net N$6: track 10.0 -> 0.00 mm
Other:
- board text added: "2022 LIGHTS"
- board text added: "On / Off"
- board text removed: "AUTHORING LIGHTS 2022"
- board text removed: "Anthony, Dave, Eric, Fred"
- board text removed: "John, Kathie, Rick"
