File: EXTENSIONS/Analog/2022.BNSK Authoring Light/bu/BNSK Authoring Light.brd (EAGLE design)
At the start: 78 x 68 mm, 22 parts

Commit message: 2022 Authoring Lights
Parts:
- moved DD1 6.32 mm to (69.0, 40.0)
- moved DE0 6.32 mm to (69.0, 54.0)
- moved DE1 6.32 mm to (69.0, 34.0)
- moved DE2 6.32 mm to (69.0, 60.0)
- moved DF0 6.32 mm to (69.0, 47.0)
- moved DF1 6.32 mm to (69.0, 28.0)
- moved DA 3.00 mm to (27.0, 69.0)
- moved DD0 3.00 mm to (60.0, 69.0)
- moved LNG_BLUE_N 2.24 mm to (35.0, 36.0)
- moved LNG_BLUE_P 2.24 mm to (50.0, 36.0)
- moved LNG_RED_N 2.24 mm to (35.0, 48.0)
- moved LNG_RED_P 2.24 mm to (50.0, 48.0)
- moved LNG_WHITE_N 2.24 mm to (35.0, 42.0)
- moved LNG_WHITE_P 2.24 mm to (50.0, 42.0)
- moved DB 1.00 mm to (38.0, 67.0)
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
Commit message: Authoring lights
Parts:
- added S1: (no value), adafruit:EG1218
- moved DD0 6.40 mm to (56.0, 64.0)
- moved DC 3.00 mm to (46.0, 65.0)
- moved DB 2.00 mm to (36.0, 67.0)
- moved DA 1.00 mm to (26.0, 69.0)
Connections:
- new net CLOCK_IN: 4017BE.14, S1.P
- net TMR555_OUTPUT: now also S1.O; no longer 4017BE.14
- net VCC: now also S1.S
Changed lines of the file:
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@@
 <attribute name="VALUE" x="17.227384375" y="50.73054375" size="1.27" layer="27" ratio="10" rot="R45"/>
 </element>
-<element name="DA" library="adafruit" package="SMADIODE" value="" x="27" y="69" smashed="yes">
-<attribute name="NAME" x="24.46" y="70.905" size="0.4064" layer="25" font="vector"/>
-<attribute name="VALUE" x="24.46" y="66.714" size="0.4064" layer="27" font="vector"/>
+<element name="DA" library="adafruit" package="SMADIODE" value="" x="26" y="69" smashed="yes">
+<attribute name="NAME" x="23.46" y="70.905" size="0.4064" layer="25" font="vector"/>
+<attribute name="VALUE" x="23.46" y="66.714" size="0.4064" layer="27" font="vector"/>
 </element>
-<element name="DB" library="adafruit" package="SMADIODE" value="" x="38" y="67" smashed="yes">
-<attribute name="NAME" x="35.46" y="68.905" size="0.4064" layer="25" font="vector"/>
-<attribute name="VALUE" x="35.46" y="64.714" size="0.4064" layer="27" font="vector"/>
+<element name="DB" library="adafruit" package="SMADIODE" value="" x="36" y="67" smashed="yes">
+<attribute name="NAME" x="33.46" y="68.905" size="0.4064" layer="25" font="vector"/>
+<attribute name="VALUE" x="33.46" y="64.714" size="0.4064" layer="27" font="vector"/>
 </element>
-<element name="DC" library="adafruit" package="SMADIODE" value="" x="49" y="65" smashed="yes">
-<attribute name="NAME" x="46.46" y="66.905" size="0.4064" layer="25" font="vector"/>
-<attribute name="VALUE" x="46.46" y="62.714" size="0.4064" layer="27" font="vector"/>
+<element name="DC" library="adafruit" package="SMADIODE" value="" x="46" y="65" smashed="yes">
+<attribute name="NAME" x="43.46" y="66.905" size="0.4064" layer="25" font="vector"/>
+<attribute name="VALUE" x="43.46" y="62.714" size="0.4064" layer="27" font="vector"/>
 </element>
-<element name="DD0" library="adafruit" package="SMADIODE" value="" x="60" y="69" smashed="yes">
-<attribute name="NAME" x="57.46" y="70.905" size="0.4064" layer="25" font="vector"/>
-<attribute name="VALUE" x="57.46" y="66.714" size="0.4064" layer="27" font="vector"/>
+<element name="DD0" library="adafruit" package="SMADIODE" value="" x="56" y="64" smashed="yes">
+<attribute name="NAME" x="53.46" y="65.905" size="0.4064" layer="25" font="vector"/>
+<attribute name="VALUE" x="53.46" y="61.714" size="0.4064" layer="27" font="vector"/>
 </element>
 <element name="DE0" library="adafruit" package="SMADIODE" value="" x="69" y="54" smashed="yes">
@@
 <attribute name="VALUE" x="66.46" y="25.714" size="0.4064" layer="27" font="vector"/>
 </element>
+<element name="S1" library="adafruit" package="EG1218" value="" x="43" y="30" smashed="yes" rot="R180">
+<attribute name="NAME" x="45.794" y="27.46" size="1.27" layer="25" font="vector" rot="R180"/>
+</element>
 </elements>
 <signals>
@@
 <contactref element="OUTPUTS" pad="2"/>
 <contactref element="4017BE" pad="16"/>
+<contactref element="S1" pad="S"/>
 <wire x1="41.23" y1="15" x2="77" y2="19.77" width="0" layer="19" extent="1-1"/>
+<wire x1="40.46" y1="30" x2="41.23" y2="15" width="0" layer="19" extent="1-1"/>
 <wire x1="24.39" y1="15.69" x2="41.23" y2="15" width="0" layer="19" extent="1-1"/>
 </signal>
@@
 <contactref element="JP_CLOCK_IN" pad="3"/>
 <contactref element="OUTPUTS" pad="3"/>
-<contactref element="4017BE" pad="14"/>
+<contactref element="S1" pad="O"/>
 <wire x1="43.77" y1="15" x2="77" y2="17.23" width="0" layer="19" extent="1-1"/>
-<wire x1="19.31" y1="15.69" x2="43.77" y2="15" width="0" layer="19" extent="1-1"/>
+<wire x1="45.54" y1="30" x2="43.77" y2="15" width="0" layer="19" extent="1-1"/>
 </signal>
 <signal name="TMR555_OUTPUT_REVERSE">
@@
 <contactref element="LED_START" pad="A"/>
 <contactref element="DA" pad="A"/>
-<wire x1="14.04" y1="76.12" x2="29.3495" y2="69" width="0" layer="19" extent="1-1"/>
-<wire x1="14.578" y1="32" x2="29.3495" y2="69" width="0" layer="19" extent="1-1"/>
+<wire x1="14.04" y1="76.12" x2="28.3495" y2="69" width="0" layer="19" extent="1-1"/>
+<wire x1="14.578" y1="32" x2="28.3495" y2="69" width="0" layer="19" extent="1-1"/>
 <wire x1="19.31" y1="23.31" x2="14.578" y2="32" width="0" layer="19" extent="1-1"/>
 </signal>
@@
 <contactref element="4017BE" pad="2"/>
 <contactref element="DB" pad="A"/>
-<wire x1="16.58" y1="76.12" x2="40.3495" y2="67" width="0" layer="19" extent="1-1"/>
-<wire x1="21.85" y1="23.31" x2="40.3495" y2="67" width="0" layer="19" extent="1-1"/>
+<wire x1="16.58" y1="76.12" x2="38.3495" y2="67" width="0" layer="19" extent="1-1"/>
+<wire x1="21.85" y1="23.31" x2="38.3495" y2="67" width="0" layer="19" extent="1-1"/>
 </signal>
 <signal name="SEG_C">
@@
 <contactref element="4017BE" pad="4"/>
 <contactref element="DC" pad="A"/>
-<wire x1="14.04" y1="60.88" x2="51.3495" y2="65" width="0" layer="19" extent="1-1"/>
+<wire x1="14.04" y1="60.88" x2="48.3495" y2="65" width="0" layer="19" extent="1-1"/>
 <wire x1="16.77" y1="23.31" x2="14.04" y2="60.88" width="0" layer="19" extent="1-1"/>
 </signal>
@@
 <contactref element="DD0" pad="A"/>
 <contactref element="DD1" pad="A"/>
-<wire x1="71.3495" y1="40" x2="62.3495" y2="69" width="0" layer="19" extent="1-1"/>
-<wire x1="8.96" y1="60.88" x2="62.3495" y2="69" width="0" layer="19" extent="1-1"/>
+<wire x1="71.3495" y1="40" x2="58.3495" y2="64" width="0" layer="19" extent="1-1"/>
+<wire x1="8.96" y1="60.88" x2="58.3495" y2="64" width="0" layer="19" extent="1-1"/>
 <wire x1="9.15" y1="23.31" x2="8.96" y2="60.88" width="0" layer="19" extent="1-1"/>
 </signal>
@@
 <wire x1="71.3495" y1="54" x2="71.3495" y2="60" width="0" layer="19" extent="1-1"/>
 <wire x1="71.3495" y1="34" x2="71.3495" y2="54" width="0" layer="19" extent="1-1"/>
-<wire x1="6.42" y1="60.88" x2="71.3495" y2="54" width="0" layer="19" extent="1-1"/>
-<wire x1="9.15" y1="15.69" x2="6.42" y2="60.88" width="0" layer="19" extent="1-1"/>
+<wire x1="9.15" y1="15.69" x2="71.3495" y2="34" width="0" layer="19" extent="1-1"/>
+<wire x1="6.42" y1="60.88" x2="9.15" y2="15.69" width="0" layer="19" extent="1-1"/>
 </signal>
 <signal name="SEG_F">
@@
 <wire x1="66.6505" y1="47" x2="66.6505" y2="54" width="0" layer="19" extent="1-1"/>
 <wire x1="50" y1="48" x2="66.6505" y2="47" width="0" layer="19" extent="1-1"/>
-<wire x1="24.6505" y1="69" x2="50" y2="48" width="0" layer="19" extent="1-1"/>
+<wire x1="23.6505" y1="69" x2="50" y2="48" width="0" layer="19" extent="1-1"/>
 </signal>
 <signal name="LNG_WHITE_P_CON">
@@
 <contactref element="DE1" pad="C"/>
 <contactref element="DF1" pad="C"/>
-<wire x1="35.6505" y1="67" x2="57.6505" y2="69" width="0" layer="19" extent="1-1"/>
-<wire x1="50" y1="42" x2="57.6505" y2="69" width="0" layer="19" extent="1-1"/>
+<wire x1="33.6505" y1="67" x2="53.6505" y2="64" width="0" layer="19" extent="1-1"/>
+<wire x1="50" y1="42" x2="53.6505" y2="64" width="0" layer="19" extent="1-1"/>
 <wire x1="66.6505" y1="34" x2="50" y2="42" width="0" layer="19" extent="1-1"/>
 <wire x1="66.6505" y1="28" x2="66.6505" y2="34" width="0" layer="19" extent="1-1"/>
@@
 <wire x1="66.6505" y1="40" x2="66.6505" y2="60" width="0" layer="19" extent="1-1"/>
 <wire x1="50" y1="36" x2="66.6505" y2="40" width="0" layer="19" extent="1-1"/>
-<wire x1="46.6505" y1="65" x2="66.6505" y2="60" width="0" layer="19" extent="1-1"/>
+<wire x1="43.6505" y1="65" x2="66.6505" y2="60" width="0" layer="19" extent="1-1"/>
+</signal>
+<signal name="CLOCK_IN">
+<contactref element="S1" pad="P"/>
+<contactref element="4017BE" pad="14"/>
+<wire x1="19.31" y1="15.69" x2="43" y2="30" width="0" layer="19" extent="1-1"/>
 </signal>
 </signals>
