File: 2023/FredT232H.Board/bu/FredT232H.Board.sch (EAGLE design)
At the start: 8 parts

Commit message: new ft232 board 2023
Connections:
- net C0: now also GPIO_OUT.10
- net C1: now also GPIO_OUT.9
- net C2: now also GPIO_OUT.8
- net C3: now also GPIO_OUT.7
- net C4: now also GPIO_OUT.6
- net C5: now also GPIO_OUT.5
- net C6: now also GPIO_OUT.4
- net C7: now also GPIO_OUT.3
- net GND: now also GPIO_OUT.1
- net VCC: now also GPIO_OUT.2
Changed lines of the file:
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@@
 <part name="GPIO_OUT" library="adafruit" deviceset="PINHD-1X10" device=""/>
 <part name="GND2" library="supply1" deviceset="GND" device=""/>
+<part name="GND5" library="supply1" deviceset="GND" device=""/>
 </parts>
 <sheets>
@@
 <attribute name="VALUE" x="-101.6" y="127" size="1.778" layer="96" rot="R90"/>
 </instance>
+<instance part="GND5" gate="1" x="5.08" y="124.46" smashed="yes" rot="R270">
+<attribute name="VALUE" x="2.54" y="127" size="1.778" layer="96" rot="R90"/>
+</instance>
 </instances>
 <busses>
@@
 <wire x1="-81.28" y1="124.46" x2="-96.52" y2="124.46" width="0.1524" layer="91"/>
 </segment>
+<segment>
+<pinref part="GPIO_OUT" gate="G$1" pin="1"/>
+<pinref part="GND5" gate="1" pin="GND"/>
+<wire x1="27.94" y1="124.46" x2="7.62" y2="124.46" width="0.1524" layer="91"/>
+</segment>
 </net>
 <net name="VCC_33" class="0">
@@
 <label x="55.88" y="109.22" size="1.778" layer="95"/>
 </segment>
+<segment>
+<pinref part="GPIO_OUT" gate="G$1" pin="3"/>
+<wire x1="27.94" y1="119.38" x2="12.7" y2="119.38" width="0.1524" layer="91"/>
+<label x="12.7" y="119.38" size="1.778" layer="95"/>
+</segment>
 </net>
 <net name="C6" class="0">
@@
 <label x="50.8" y="111.76" size="1.778" layer="95"/>
 </segment>
+<segment>
+<pinref part="GPIO_OUT" gate="G$1" pin="4"/>
+<wire x1="27.94" y1="116.84" x2="7.62" y2="116.84" width="0.1524" layer="91"/>
+<label x="12.7" y="116.84" size="1.778" layer="95"/>
+</segment>
 </net>
 <net name="C5" class="0">
@@
 <label x="53.34" y="114.3" size="1.778" layer="95"/>
 </segment>
+<segment>
+<pinref part="GPIO_OUT" gate="G$1" pin="5"/>
+<wire x1="27.94" y1="114.3" x2="15.24" y2="114.3" width="0.1524" layer="91"/>
+<label x="15.24" y="114.3" size="1.778" layer="95"/>
+</segment>
 </net>
 <net name="C4" class="0">
@@
 <label x="48.26" y="116.84" size="1.778" layer="95"/>
 </segment>
+<segment>
+<pinref part="GPIO_OUT" gate="G$1" pin="6"/>
+<wire x1="27.94" y1="111.76" x2="7.62" y2="111.76" width="0.1524" layer="91"/>
+<label x="12.7" y="111.76" size="1.778" layer="95"/>
+</segment>
 </net>
 <net name="C3" class="0">
@@
 <label x="55.88" y="119.38" size="1.778" layer="95"/>
 </segment>
+<segment>
+<pinref part="GPIO_OUT" gate="G$1" pin="7"/>
+<wire x1="27.94" y1="109.22" x2="10.16" y2="109.22" width="0.1524" layer="91"/>
+<label x="12.7" y="109.22" size="1.778" layer="95"/>
+</segment>
 </net>
 <net name="C2" class="0">
@@
 <label x="48.26" y="121.92" size="1.778" layer="95"/>
 </segment>
+<segment>
+<pinref part="GPIO_OUT" gate="G$1" pin="8"/>
+<wire x1="27.94" y1="106.68" x2="5.08" y2="106.68" width="0.1524" layer="91"/>
+<label x="12.7" y="106.68" size="1.778" layer="95"/>
+</segment>
 </net>
 <net name="C1" class="0">
@@
 <label x="58.42" y="124.46" size="1.778" layer="95"/>
 </segment>
+<segment>
+<pinref part="GPIO_OUT" gate="G$1" pin="9"/>
+<wire x1="27.94" y1="104.14" x2="12.7" y2="104.14" width="0.1524" layer="91"/>
+<label x="17.78" y="104.14" size="1.778" layer="95"/>
+</segment>
 </net>
 <net name="C0" class="0">
@@
 <wire x1="68.58" y1="127" x2="48.26" y2="127" width="0.1524" layer="91"/>
 <label x="50.8" y="127" size="1.778" layer="95"/>
+</segment>
+<segment>
+<pinref part="GPIO_OUT" gate="G$1" pin="10"/>
+<wire x1="27.94" y1="101.6" x2="7.62" y2="101.6" width="0.1524" layer="91"/>
+<label x="10.16" y="101.6" size="1.778" layer="95"/>
 </segment>
 </net>
@@
 <label x="-96.52" y="121.92" size="1.778" layer="95"/>
 </segment>
-</net>
+<segment>
+<pinref part="GPIO_OUT" gate="G$1" pin="2"/>
+<wire x1="27.94" y1="121.92" x2="7.62" y2="121.92" width="0.1524" layer="91"/>
+<label x="10.16" y="121.92" size="1.778" layer="95"/>
+</segment>
+</net>
