File: 2023/Nusbio Thumb Drive/bu/Ex EEPROM.sch (EAGLE design)
At the start: 8 parts

Commit message: new ft232 board 2023
Parts:
- removed GPIO_OUT, SPI_OUT: PINHD-1X10, adafruit:PINHD-1X10
- removed JP_GPIO, JP_SPI: (no value), pinhead:PINHD-1X11
- removed LED_POWER: (no value), adafruit:LEDSMT1206
- removed R_1K: (no value), adafruit:R-US_R1206
- removed VCC_33, VCC_5V: (no value), microbuilder:SOLDERJUMPERREFLOW
- added NUSBIO_IN, NUSBIO_OUT: PINHD-1X10, adafruit:PINHD-1X10
- added R1: (no value), adafruit:R-US_R1206
- added SPI_SOIC_FLASH: 25AA080SN, microchip:25AA080SN
- added WRITE_ENABLE: (no value), microbuilder:SOLDERJUMPERREFLOW
Connections:
- removed net C0: GPIO_OUT.10, JP_GPIO.1
- removed net C1: GPIO_OUT.9, JP_GPIO.2
- removed net C2: GPIO_OUT.8, JP_GPIO.3
- removed net C3: GPIO_OUT.7, JP_GPIO.4
- removed net C4: GPIO_OUT.6, JP_GPIO.5
- removed net C5: GPIO_OUT.5, JP_GPIO.6
- removed net C6: GPIO_OUT.4, JP_GPIO.7
- removed net C7: GPIO_OUT.3, JP_GPIO.8
- removed net D0_SCLK: JP_SPI.8, SPI_OUT.10
- removed net D1_MOSI: JP_SPI.7, SPI_OUT.9
- removed net D2_MISO: JP_SPI.6, SPI_OUT.8
- removed net D3_CS0: JP_SPI.5, SPI_OUT.7
- removed net D4_CS1: JP_SPI.4, SPI_OUT.6
- removed net D5_CS2: JP_SPI.3, SPI_OUT.5
- removed net D6_CS3: JP_SPI.2, SPI_OUT.4
- removed net D7_CS4: JP_SPI.1, SPI_OUT.3
- removed net VCC_33: JP_SPI.11, VCC_33.2
- removed net VCC_5: JP_SPI.10, LED_POWER.A, VCC_5V.2
- new net CS: NUSBIO_IN.4, NUSBIO_OUT.4, SPI_SOIC_FLASH.!CS
- new net GPIO5: NUSBIO_IN.5, NUSBIO_OUT.5
- new net GPIO6: NUSBIO_IN.6, NUSBIO_OUT.6
- new net GPIO7: NUSBIO_IN.7, NUSBIO_OUT.7
- new net GPIO8: NUSBIO_IN.8, NUSBIO_OUT.8
- new net MISO: NUSBIO_IN.3, NUSBIO_OUT.3, SPI_SOIC_FLASH.SO
- new net MOSI: NUSBIO_IN.2, NUSBIO_OUT.2, SPI_SOIC_FLASH.SI
- new net SCK: NUSBIO_IN.1, NUSBIO_OUT.1, SPI_SOIC_FLASH.SCK
- net GND: now also NUSBIO_IN.10, NUSBIO_OUT.10, SPI_SOIC_FLASH.GND; no longer GPIO_OUT.1, JP_GPIO.11, JP_SPI.9, R_1K.1, SPI_OUT.1
- net N$1: now also SPI_SOIC_FLASH.!WP, WRITE_ENABLE.2; no longer LED_POWER.C, R_1K.2
- net VCC: now also NUSBIO_IN.9, NUSBIO_OUT.9, SPI_SOIC_FLASH.!HOLD, SPI_SOIC_FLASH.VCC, WRITE_ENABLE.1; no longer GPIO_OUT.2, SPI_OUT.2, VCC_33.1, VCC_5V.1
