File: 2023/Nusbio Flash Extension/Nusbio Flash Extension.brd (EAGLE design)
At the start: 44 x 50 mm, 8 parts

Commit message: fDrive update
Parts:
- removed NUSBIO_IN: PINHD-1X10, adafruit:1X10-BIG
- added GPIO_IN: PINHD-1X10, adafruit:1X10-BIG
- moved LED_POWER 3.39 mm to (39.9, 37.8)
- moved SPI_SOIC_8_FLASH 1.12 mm to (21.5, 20.0)
- moved R_1K 0.50 mm to (38.0, 27.5)
- renumbered NUSBIO_OUT to GPIO_OUT
Connections:
- net CS_4: now also GPIO_IN.4; no longer NUSBIO_IN.4
- net CS_5: now also GPIO_IN.5; no longer NUSBIO_IN.5
- net GND: now also GPIO_IN.10; no longer NUSBIO_IN.10
- net GPIO6: now also GPIO_IN.6; no longer NUSBIO_IN.6
- net GPIO7: now also GPIO_IN.7; no longer NUSBIO_IN.7
- net GPIO8: now also GPIO_IN.8; no longer NUSBIO_IN.8
- net MISO: now also GPIO_IN.3; no longer NUSBIO_IN.3
- net MOSI: now also GPIO_IN.2; no longer NUSBIO_IN.2
- net SCK: now also GPIO_IN.1; no longer NUSBIO_IN.1
- net VCC: now also GPIO_IN.9; no longer NUSBIO_IN.9
Other:
- board text added: "C:/DVT/Fred.PCB/2023/MadeInTheUSB.Logo.Gray.50.bmp"
- board text added: "C:/DVT/Fred.PCB/2023/Nusbio Flash Extension/MadeInTheUSB.Logo.Gray.bmp"
- board text added: "C:/DVT/Fred.PCB/2023/Nusbio Flash Extension/Title.Logo.Gray.bmp"
- board text removed: "Flash Extension"

Commit message: update
Parts:
- removed WRITE_DISABLE: (no value), microbuilder:SOLDERJUMPER_REFLOW
Connections:
- removed net WP: SPI_SOIC_8_FLASH.3, WRITE_DISABLE.2
- net GND: no longer WRITE_DISABLE.1
- net VCC: now also SPI_SOIC_8_FLASH.3
Changed lines of the file:
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@@
 <attribute name="OC_NEWARK" value="92C7351" x="21.5" y="20" size="1.778" layer="27" rot="R270" display="off"/>
-</element>
-<element name="WRITE_DISABLE" library="microbuilder" package="SOLDERJUMPER_REFLOW" value="" x="7" y="21.5" smashed="yes" rot="R90">
-<attribute name="NAME" x="5" y="21" size="0.8128" layer="25" ratio="18" rot="R90" align="center"/>
-<attribute name="VALUE" x="7" y="21.9001" size="0.02" layer="27" rot="R90"/>
 </element>
 <element name="R_1K" library="adafruit" package="R1206" value="" x="38" y="27.5" smashed="yes">
@@
 <contactref element="SPI_SOIC_8_FLASH" pad="4"/>
 <contactref element="R_1K" pad="1"/>
-<contactref element="WRITE_DISABLE" pad="1"/>
 <wire x1="18.9" y1="18.095" x2="36.578" y2="27.5" width="0" layer="19" extent="1-1"/>
-<wire x1="7" y1="20.738" x2="18.9" y2="18.095" width="0" layer="19" extent="1-1"/>
 <wire x1="33.782071875" y1="2.37569375" x2="18.9" y2="18.095" width="0" layer="19" extent="1-1"/>
-<wire x1="10.9" y1="48" x2="7" y2="20.738" width="0" layer="19" extent="1-1"/>
+<wire x1="10.9" y1="48" x2="18.9" y2="18.095" width="0" layer="19" extent="1-1"/>
 </signal>
 <signal name="VCC">
@@
 <contactref element="SPI_SOIC_8_FLASH" pad="7"/>
 <contactref element="LED_POWER" pad="A"/>
+<contactref element="SPI_SOIC_8_FLASH" pad="3"/>
 <wire x1="24.1" y1="21.905" x2="38.467" y2="37.8095" width="0" layer="19" extent="1-1"/>
 <wire x1="24.1" y1="20.635" x2="24.1" y2="21.905" width="0" layer="19" extent="1-1"/>
+<wire x1="18.9" y1="19.365" x2="24.1" y2="20.635" width="0" layer="19" extent="1-1"/>
 <wire x1="31.242071875" y1="2.37569375" x2="24.1" y2="20.635" width="0" layer="19" extent="1-1"/>
 <wire x1="13.44" y1="48" x2="38.467" y2="37.8095" width="0" layer="19" extent="1-1"/>
@@
 <wire x1="18.9" y1="21.905" x2="38.762" y2="20" width="0" layer="19" extent="1-1"/>
 </signal>
-<signal name="WP">
-<contactref element="WRITE_DISABLE" pad="2"/>
-<contactref element="SPI_SOIC_8_FLASH" pad="3"/>
-<wire x1="7" y1="22.262" x2="18.9" y2="19.365" width="0" layer="19" extent="1-1"/>
-</signal>
 <signal name="GPIO6">
