File: 2023/Nusbio Flash Extension/Nusbio Flash Extension.sch (EAGLE design)
At the start: 8 parts

Commit message: fDrive update
Parts:
- renumbered NUSBIO_IN to GPIO_IN, NUSBIO_OUT to GPIO_OUT
Changed lines of the file:
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@@
 </classes>
 <parts>
-<part name="NUSBIO_IN" library="adafruit" deviceset="PINHD-1X10" device=""/>
+<part name="GPIO_IN" library="adafruit" deviceset="PINHD-1X10" device=""/>
 <part name="GND1" library="supply1" deviceset="GND" device=""/>
-<part name="NUSBIO_OUT" library="adafruit" deviceset="PINHD-1X10" device=""/>
+<part name="GPIO_OUT" library="adafruit" deviceset="PINHD-1X10" device=""/>
 <part name="GND3" library="supply1" deviceset="GND" device=""/>
 <part name="SPI_SOIC_8_FLASH" library="microchip" deviceset="25*" device="SN" technology="AA080"/>
@@
 </plain>
 <instances>
-<instance part="NUSBIO_IN" gate="G$1" x="17.78" y="55.88" smashed="yes" rot="R180">
+<instance part="GPIO_IN" gate="G$1" x="17.78" y="55.88" smashed="yes" rot="R180">
 <attribute name="NAME" x="24.13" y="42.545" size="1.778" layer="95" rot="R180"/>
 </instance>
@@
 <attribute name="VALUE" x="10.16" y="73.66" size="1.778" layer="96" rot="R90"/>
 </instance>
-<instance part="NUSBIO_OUT" gate="G$1" x="99.06" y="55.88" smashed="yes">
+<instance part="GPIO_OUT" gate="G$1" x="99.06" y="55.88" smashed="yes">
 <attribute name="NAME" x="92.71" y="69.215" size="1.778" layer="95"/>
 </instance>
@@
 <segment>
 <pinref part="GND1" gate="1" pin="GND"/>
-<pinref part="NUSBIO_IN" gate="G$1" pin="10"/>
+<pinref part="GPIO_IN" gate="G$1" pin="10"/>
 <wire x1="5.08" y1="76.2" x2="20.32" y2="68.58" width="0.1524" layer="91"/>
 </segment>
 <segment>
 <pinref part="GND3" gate="1" pin="GND"/>
-<pinref part="NUSBIO_OUT" gate="G$1" pin="10"/>
+<pinref part="GPIO_OUT" gate="G$1" pin="10"/>
 <wire x1="66.04" y1="43.18" x2="96.52" y2="43.18" width="0.1524" layer="91"/>
 </segment>
@@
 <net name="VCC" class="0">
 <segment>
-<pinref part="NUSBIO_IN" gate="G$1" pin="9"/>
+<pinref part="GPIO_IN" gate="G$1" pin="9"/>
 <wire x1="20.32" y1="66.04" x2="30.48" y2="66.04" width="0.1524" layer="91"/>
 <label x="27.94" y="68.58" size="1.778" layer="95"/>
 </segment>
 <segment>
-<pinref part="NUSBIO_OUT" gate="G$1" pin="9"/>
+<pinref part="GPIO_OUT" gate="G$1" pin="9"/>
 <wire x1="96.52" y1="45.72" x2="87.376" y2="45.72" width="0.1524" layer="91"/>
 <label x="82.296" y="45.72" size="1.778" layer="95"/>
@@
 <net name="SCK" class="0">
 <segment>
-<pinref part="NUSBIO_IN" gate="G$1" pin="1"/>
+<pinref part="GPIO_IN" gate="G$1" pin="1"/>
 <wire x1="20.32" y1="45.72" x2="27.94" y2="45.72" width="0.1524" layer="91"/>
 <label x="27.94" y="45.72" size="1.778" layer="95"/>
@@
 </segment>
 <segment>
-<pinref part="NUSBIO_OUT" gate="G$1" pin="1"/>
+<pinref part="GPIO_OUT" gate="G$1" pin="1"/>
 <wire x1="96.52" y1="66.04" x2="84.582" y2="66.04" width="0.1524" layer="91"/>
 <label x="82.042" y="66.04" size="1.778" layer="95"/>
@@
 <net name="MOSI" class="0">
 <segment>
-<pinref part="NUSBIO_IN" gate="G$1" pin="2"/>
+<pinref part="GPIO_IN" gate="G$1" pin="2"/>
 <wire x1="20.32" y1="48.26" x2="27.94" y2="48.26" width="0.1524" layer="91"/>
 <label x="27.94" y="48.26" size="1.778" layer="95"/>
@@
 </segment>
 <segment>
-<pinref part="NUSBIO_OUT" gate="G$1" pin="2"/>
+<pinref part="GPIO_OUT" gate="G$1" pin="2"/>
 <wire x1="96.52" y1="63.5" x2="84.582" y2="63.5" width="0.1524" layer="91"/>
 <label x="82.042" y="63.5" size="1.778" layer="95"/>
@@
 <net name="MISO" class="0">
 <segment>
-<pinref part="NUSBIO_IN" gate="G$1" pin="3"/>
+<pinref part="GPIO_IN" gate="G$1" pin="3"/>
 <wire x1="20.32" y1="50.8" x2="27.94" y2="50.8" width="0.1524" layer="91"/>
 <label x="27.94" y="50.8" size="1.778" layer="95"/>
@@
 </segment>
 <segment>
-<pinref part="NUSBIO_OUT" gate="G$1" pin="3"/>
+<pinref part="GPIO_OUT" gate="G$1" pin="3"/>
 <wire x1="96.52" y1="60.96" x2="84.582" y2="60.96" width="0.1524" layer="91"/>
 <label x="82.042" y="60.96" size="1.778" layer="95"/>
@@
 <net name="GPIO6" class="0">
 <segment>
-<pinref part="NUSBIO_OUT" gate="G$1" pin="6"/>
+<pinref part="GPIO_OUT" gate="G$1" pin="6"/>
 <wire x1="96.52" y1="53.34" x2="86.36" y2="53.34" width="0.1524" layer="91"/>
 <label x="83.82" y="53.34" size="1.778" layer="95"/>
 </segment>
 <segment>
-<pinref part="NUSBIO_IN" gate="G$1" pin="6"/>
+<pinref part="GPIO_IN" gate="G$1" pin="6"/>
 <wire x1="20.32" y1="58.42" x2="27.94" y2="58.42" width="0.1524" layer="91"/>
 <label x="27.94" y="58.42" size="1.778" layer="95"/>
@@
 <net name="GPIO7" class="0">
 <segment>
-<pinref part="NUSBIO_IN" gate="G$1" pin="7"/>
+<pinref part="GPIO_IN" gate="G$1" pin="7"/>
 <wire x1="20.32" y1="60.96" x2="27.94" y2="60.96" width="0.1524" layer="91"/>
 <label x="27.94" y="60.96" size="1.778" layer="95"/>
 </segment>
 <segment>
-<pinref part="NUSBIO_OUT" gate="G$1" pin="7"/>
+<pinref part="GPIO_OUT" gate="G$1" pin="7"/>
 <wire x1="96.52" y1="50.8" x2="86.36" y2="50.8" width="0.1524" layer="91"/>
 <label x="86.36" y="50.8" size="1.778" layer="95"/>
@@
 <net name="GPIO8" class="0">
 <segment>
-<pinref part="NUSBIO_IN" gate="G$1" pin="8"/>
+<pinref part="GPIO_IN" gate="G$1" pin="8"/>
 <wire x1="20.32" y1="63.5" x2="27.94" y2="63.5" width="0.1524" layer="91"/>
 <label x="27.94" y="63.5" size="1.778" layer="95"/>
 </segment>
 <segment>
-<pinref part="NUSBIO_OUT" gate="G$1" pin="8"/>
+<pinref part="GPIO_OUT" gate="G$1" pin="8"/>
 <wire x1="96.52" y1="48.26" x2="86.36" y2="48.26" width="0.1524" layer="91"/>
 <label x="86.36" y="48.26" size="1.778" layer="95"/>
@@
 <net name="CS_4" class="0">
 <segment>
-<pinref part="NUSBIO_IN" gate="G$1" pin="4"/>
+<pinref part="GPIO_IN" gate="G$1" pin="4"/>
 <wire x1="20.32" y1="53.34" x2="25.4" y2="53.34" width="0.1524" layer="91"/>
 <wire x1="25.4" y1="53.34" x2="27.94" y2="53.34" width="0.1524" layer="91"/>
@@
 </segment>
 <segment>
-<pinref part="NUSBIO_OUT" gate="G$1" pin="4"/>
+<pinref part="GPIO_OUT" gate="G$1" pin="4"/>
 <wire x1="96.52" y1="58.42" x2="84.582" y2="58.42" width="0.1524" layer="91"/>
 <label x="82.042" y="58.42" size="1.778" layer="95"/>
@@
 <net name="CS_5" class="0">
 <segment>
-<pinref part="NUSBIO_IN" gate="G$1" pin="5"/>
+<pinref part="GPIO_IN" gate="G$1" pin="5"/>
 <wire x1="20.32" y1="55.88" x2="27.94" y2="55.88" width="0.1524" layer="91"/>
 <label x="27.94" y="55.88" size="1.778" layer="95"/>
@@
 </segment>
 <segment>
-<pinref part="NUSBIO_OUT" gate="G$1" pin="5"/>
+<pinref part="GPIO_OUT" gate="G$1" pin="5"/>
 <wire x1="96.52" y1="55.88" x2="86.36" y2="55.88" width="0.1524" layer="91"/>
 <label x="81.28" y="55.88" size="1.778" layer="95"/>

Commit message: update
Parts:
- removed WRITE_DISABLE: (no value), microbuilder:SOLDERJUMPERREFLOW
Connections:
- removed net WP: SPI_SOIC_8_FLASH.!WP, WRITE_DISABLE.2
- net GND: no longer WRITE_DISABLE.1
- net VCC: now also SPI_SOIC_8_FLASH.!WP
Changed lines of the file:
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@@
 <part name="SPI_SOIC_8_FLASH" library="microchip" deviceset="25*" device="SN" technology="AA080"/>
 <part name="GND2" library="supply1" deviceset="GND" device=""/>
-<part name="WRITE_DISABLE" library="microbuilder" deviceset="SOLDERJUMPER" device="REFLOW"/>
 <part name="R_1K" library="adafruit" deviceset="R-US_" device="R1206"/>
 <part name="LED_POWER" library="adafruit" deviceset="LED" device="SMT1206"/>
@@
 <part name="USE_CS_3" library="microbuilder" deviceset="SOLDERJUMPER" device="REFLOW"/>
 <part name="USE_CS_4" library="microbuilder" deviceset="SOLDERJUMPER" device="REFLOW"/>
-<part name="GND5" library="supply1" deviceset="GND" device=""/>
 </parts>
 <sheets>
@@
 <attribute name="VALUE" x="66.04" y="50.8" size="1.778" layer="96" rot="MR0"/>
 </instance>
-<instance part="WRITE_DISABLE" gate="1" x="35.56" y="76.2" smashed="yes">
-<attribute name="NAME" x="33.02" y="78.74" size="1.778" layer="95"/>
-<attribute name="VALUE" x="33.02" y="72.39" size="1.778" layer="96"/>
-</instance>
 <instance part="R_1K" gate="G$1" x="93.98" y="93.98" smashed="yes">
 <attribute name="NAME" x="90.17" y="95.4786" size="1.778" layer="95"/>
@@
 <attribute name="NAME" x="17.78" y="99.06" size="1.778" layer="95"/>
 <attribute name="VALUE" x="17.78" y="92.71" size="1.778" layer="96"/>
-</instance>
-<instance part="GND5" gate="1" x="17.78" y="76.2" smashed="yes" rot="R270">
-<attribute name="VALUE" x="15.24" y="78.74" size="1.778" layer="96" rot="R270"/>
 </instance>
 </instances>
@@
 <wire x1="88.9" y1="93.98" x2="81.28" y2="93.98" width="0.1524" layer="91"/>
 </segment>
-<segment>
-<pinref part="GND5" gate="1" pin="GND"/>
-<pinref part="WRITE_DISABLE" gate="1" pin="1"/>
-<wire x1="20.32" y1="76.2" x2="30.48" y2="76.2" width="0.1524" layer="91"/>
-</segment>
 </net>
 <net name="VCC" class="0">
@@
 <pinref part="LED_POWER" gate="G$1" pin="A"/>
 <wire x1="114.3" y1="93.98" x2="127" y2="93.98" width="0.1524" layer="91"/>
+</segment>
+<segment>
+<pinref part="SPI_SOIC_8_FLASH" gate="G$1" pin="!WP"/>
+<wire x1="43.18" y1="76.2" x2="30.48" y2="76.2" width="0.1524" layer="91"/>
+<label x="30.48" y="78.74" size="1.778" layer="95"/>
 </segment>
 </net>
@@
 </segment>
 </net>
-<net name="WP" class="0">
-<segment>
-<pinref part="WRITE_DISABLE" gate="1" pin="2"/>
-<pinref part="SPI_SOIC_8_FLASH" gate="G$1" pin="!WP"/>
-<wire x1="40.64" y1="76.2" x2="43.18" y2="76.2" width="0.1524" layer="91"/>
-<label x="40.64" y="76.2" size="1.778" layer="95"/>
-</segment>
-</net>

Commit message: update from 2023.03
Parts:
- renumbered R_1K to R_4K
Connections:
- removed net CS_5: GPIO_IN.5, GPIO_OUT.5, USE_CS_4.1
- new net CS_3: GPIO_IN.4, GPIO_OUT.4, USE_CS_3.1
- net CS_4: now also GPIO_IN.5, GPIO_OUT.5, USE_CS_4.1; no longer GPIO_IN.4, GPIO_OUT.4, USE_CS_3.1
Changed lines of the file:
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@@
 <part name="SPI_SOIC_8_FLASH" library="microchip" deviceset="25*" device="SN" technology="AA080"/>
 <part name="GND2" library="supply1" deviceset="GND" device=""/>
-<part name="R_1K" library="adafruit" deviceset="R-US_" device="R1206"/>
+<part name="R_4K" library="adafruit" deviceset="R-US_" device="R1206"/>
 <part name="LED_POWER" library="adafruit" deviceset="LED" device="SMT1206"/>
 <part name="GND4" library="supply1" deviceset="GND" device=""/>
@@
 <attribute name="NAME" x="24.13" y="42.545" size="1.778" layer="95" rot="R180"/>
 </instance>
-<instance part="GND1" gate="1" x="7.62" y="76.2" smashed="yes" rot="R90">
-<attribute name="VALUE" x="10.16" y="73.66" size="1.778" layer="96" rot="R90"/>
+<instance part="GND1" gate="1" x="20.32" y="81.28" smashed="yes" rot="R180">
+<attribute name="VALUE" x="27.94" y="83.82" size="1.778" layer="96" rot="R180"/>
 </instance>
 <instance part="GPIO_OUT" gate="G$1" x="99.06" y="55.88" smashed="yes">
@@
 <attribute name="VALUE" x="66.04" y="50.8" size="1.778" layer="96" rot="MR0"/>
 </instance>
-<instance part="R_1K" gate="G$1" x="93.98" y="93.98" smashed="yes">
+<instance part="R_4K" gate="G$1" x="93.98" y="93.98" smashed="yes">
 <attribute name="NAME" x="90.17" y="95.4786" size="1.778" layer="95"/>
 <attribute name="VALUE" x="90.17" y="90.678" size="1.778" layer="96"/>
@@
 <pinref part="GND1" gate="1" pin="GND"/>
 <pinref part="GPIO_IN" gate="G$1" pin="10"/>
-<wire x1="5.08" y1="76.2" x2="20.32" y2="68.58" width="0.1524" layer="91"/>
+<wire x1="20.32" y1="78.74" x2="20.32" y2="68.58" width="0.1524" layer="91"/>
 </segment>
 <segment>
@@
 </segment>
 <segment>
-<pinref part="R_1K" gate="G$1" pin="1"/>
+<pinref part="R_4K" gate="G$1" pin="1"/>
 <pinref part="GND4" gate="1" pin="GND"/>
 <wire x1="88.9" y1="93.98" x2="81.28" y2="93.98" width="0.1524" layer="91"/>
@@
 <segment>
 <pinref part="LED_POWER" gate="G$1" pin="C"/>
-<pinref part="R_1K" gate="G$1" pin="2"/>
+<pinref part="R_4K" gate="G$1" pin="2"/>
 <wire x1="106.68" y1="93.98" x2="99.06" y2="93.98" width="0.1524" layer="91"/>
 </segment>
 </net>
 <net name="CS_4" class="0">
+<segment>
+<pinref part="GPIO_IN" gate="G$1" pin="5"/>
+<wire x1="20.32" y1="55.88" x2="27.94" y2="55.88" width="0.1524" layer="91"/>
+<label x="27.94" y="55.88" size="1.778" layer="95"/>
+</segment>
+<segment>
+<pinref part="GPIO_OUT" gate="G$1" pin="5"/>
+<wire x1="96.52" y1="55.88" x2="86.36" y2="55.88" width="0.1524" layer="91"/>
+<label x="81.28" y="55.88" size="1.778" layer="95"/>
+</segment>
+<segment>
+<pinref part="USE_CS_4" gate="1" pin="1"/>
+<wire x1="15.24" y1="96.52" x2="5.08" y2="96.52" width="0.1524" layer="91"/>
+</segment>
+</net>
+<net name="CS_3" class="0">
 <segment>
 <pinref part="GPIO_IN" gate="G$1" pin="4"/>
@@
 </segment>
 <segment>
-<pinref part="USE_CS_3" gate="1" pin="1"/>
-<wire x1="15.24" y1="104.14" x2="5.08" y2="104.14" width="0.1524" layer="91"/>
-<label x="5.08" y="101.6" size="1.778" layer="95"/>
-</segment>
-<segment>
 <pinref part="GPIO_OUT" gate="G$1" pin="4"/>
 <wire x1="96.52" y1="58.42" x2="84.582" y2="58.42" width="0.1524" layer="91"/>
 <label x="82.042" y="58.42" size="1.778" layer="95"/>
 </segment>
-</net>
-<net name="CS_5" class="0">
-<segment>
-<pinref part="GPIO_IN" gate="G$1" pin="5"/>
-<wire x1="20.32" y1="55.88" x2="27.94" y2="55.88" width="0.1524" layer="91"/>
-<label x="27.94" y="55.88" size="1.778" layer="95"/>
-</segment>
-<segment>
-<pinref part="USE_CS_4" gate="1" pin="1"/>
-<wire x1="15.24" y1="96.52" x2="5.08" y2="96.52" width="0.1524" layer="91"/>
-</segment>
-<segment>
-<pinref part="GPIO_OUT" gate="G$1" pin="5"/>
-<wire x1="96.52" y1="55.88" x2="86.36" y2="55.88" width="0.1524" layer="91"/>
-<label x="81.28" y="55.88" size="1.778" layer="95"/>
-</segment>
-</net>
+<segment>
+<pinref part="USE_CS_3" gate="1" pin="1"/>
+<wire x1="15.24" y1="104.14" x2="5.08" y2="104.14" width="0.1524" layer="91"/>
+<label x="5.08" y="106.68" size="1.778" layer="95"/>
+</segment>
+</net>
