File: 2023/BNSK-Rambo-Converters-Device/bu/BNSK-Rambo-Converters-Device.brd (EAGLE design)
At the start: 68 x 58 mm, 9 parts

Commit message: 2023.2. PCBs
Parts:
- removed CHECKING: (no value), adafruit:1206
- moved R_ARRAY_8 1.87 mm to (5.81, 42.6), turned to 270 degrees
Connections:
- net MCU_D4: no longer CHECKING.A
- net RA_6: no longer CHECKING.C
Other:
- board text added: "C:/DVT/Fred.PCB/2023/BNSK-Rambo-Converters-Device/Title.Converters Automation Device.bmp"
- board text added: "C:/DVT/Fred.PCB/2023/BNSK-Rambo-Converters-Device/Title.fDrive.Logo.Gray.bmp"
- board text added: "XIAO ESP32 C3"
- board text removed: "Converters Automation Device"
- board text removed: "RAMBO"
