File: 2023/FredT232H.Board/v1/FredT232H.Board.brd (EAGLE design)
At the start: 88 x 77 mm, 17 parts

Commit message: 2023.2. PCBs
Routing:
- net GND: track 233.4 -> 0.00 mm, vias 2 -> 0
- net VCC_33: track 168.6 -> 0.00 mm
- net D3_CS0: track 144.7 -> 0.00 mm
- net D4_CS1: track 108.8 -> 0.00 mm, vias 1 -> 0
- net D1_MOSI: track 107.8 -> 0.00 mm
- net D7_CS4: track 107.1 -> 0.00 mm, vias 1 -> 0
- net C4: track 105.8 -> 0.00 mm
- net D5_CS2: track 105.2 -> 0.00 mm, vias 1 -> 0
- net C7: track 103.8 -> 0.00 mm
- net D6_CS3: track 101.3 -> 0.00 mm, vias 2 -> 0
- net D2_MISO: track 99.5 -> 0.00 mm, vias 1 -> 0
- net D0_SCLK: track 98.9 -> 0.00 mm
- net C6: track 98.3 -> 0.00 mm
- net C5: track 92.8 -> 0.00 mm
- net C3: track 82.2 -> 0.00 mm
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