File: 2023/Nusbio Flash Extension/v1/Nusbio Flash Extension.brd (EAGLE design)
At the start: 44 x 50 mm, 7 parts

Commit message: 2023.2. PCBs
Routing:
- net GND: track 87.5 -> 0.00 mm, vias 1 -> 0
- net VCC: track 86.2 -> 0.00 mm, vias 2 -> 0
- net CS_4: track 77.6 -> 0.00 mm
- net CS_5: track 62.5 -> 0.00 mm, vias 2 -> 0
- net MISO: track 58.0 -> 0.00 mm, vias 2 -> 0
- net SCK: track 57.7 -> 0.00 mm, vias 1 -> 0
- net MOSI: track 55.2 -> 0.00 mm, vias 1 -> 0
- net GPIO8: track 52.7 -> 0.00 mm, vias 1 -> 0
- net GPIO7: track 50.3 -> 0.00 mm, vias 1 -> 0
- net GPIO6: track 46.9 -> 0.00 mm
- net CS: track 29.6 -> 0.00 mm
- net N$2: track 11.4 -> 0.00 mm
