File: 2023/USB Experiment Board/v1/USB Experiment Board.sch (EAGLE design)
At the start: 8 parts

Commit message: 2023.2. PCBs
Parts:
- removed CHECK_NOW: (no value), switch-omron:10-XX
- removed FAILED, PASSED, RUNNING: (no value), adafruit:LEDSMT1206
- removed MCU_LEFT_SIDE, MCU_RIGHT_SIDE: (no value), pinhead:PINHD-1X7
- removed R_ARRAY_8: (no value), adafruit:PINHD-1X9
- added BB_1, BB_10, BB_11, BB_12, BB_13, BB_14, BB_15, BB_16, BB_17, BB_18, BB_19, BB_2, BB_20, BB_3, BB_4, BB_5, BB_6, BB_7, BB_8, BB_9, GND_RAIL_L, GND_RAIL_R, R_ARRAY_2_CON, VCC_RAIL_L, VCC_RAIL_R: PINHD-1X10, adafruit:PINHD-1X10
- added BUTTON_1_SYNC, BUTTON_2: (no value), switch-omron:10-XX
- added BUTTON_INPUTS, JP_DTA: (no value), pinhead:PINHD-1X2
- added LED1, LED2, LED3, LED4: (no value), adafruit:LEDSMT1206
- added LED_HEADER: (no value), pinhead:PINHD-1X4
- added R_ARRAY_1, R_ARRAY_2: (no value), resistor-sip:4610X
- added U$1: USB, STUNTAZ:USB
- added X1: USB-A, adafruit:USB-A
Connections:
- removed net MCU_D0: MCU_RIGHT_SIDE.1, PASSED.A
- removed net MCU_D1: FAILED.A, MCU_RIGHT_SIDE.2
- removed net MCU_D10: MCU_LEFT_SIDE.4
- removed net MCU_D2: MCU_RIGHT_SIDE.3, RUNNING.A
- removed net MCU_D3: CHECK_NOW.S, MCU_RIGHT_SIDE.4
- removed net MCU_D4: MCU_RIGHT_SIDE.5
- removed net MCU_D5: MCU_RIGHT_SIDE.6
- removed net MCU_D6: MCU_RIGHT_SIDE.7
- removed net MCU_D7: MCU_LEFT_SIDE.1
- removed net MCU_D8: MCU_LEFT_SIDE.2
- removed net MCU_D9: MCU_LEFT_SIDE.3
- removed net MCU_VCC_5V: MCU_LEFT_SIDE.7
- removed net RA_1: POWER.C, R_ARRAY_8.2
- removed net RA_2: PASSED.C, R_ARRAY_8.3
- removed net RA_3: FAILED.C, R_ARRAY_8.4
- removed net RA_4: RUNNING.C, R_ARRAY_8.5
- removed net RA_5: CHECK_NOW.P1, R_ARRAY_8.6
- removed net RA_6: R_ARRAY_8.7
- removed net VCC_33: MCU_LEFT_SIDE.5, POWER.A
- new net B1_INPUT: BUTTON_1_SYNC.S, BUTTON_INPUTS.1
- new net B2_OUTPUT: BUTTON_2.P1, BUTTON_INPUTS.2
- new net N$1: R_ARRAY_2.2, R_ARRAY_2_CON.10
- new net N$10: LED3.A, LED_HEADER.3
- new net N$11: LED4.A, LED_HEADER.4
- new net N$12: R_ARRAY_2.3, R_ARRAY_2_CON.9
- new net N$13: POWER.C, R_ARRAY_1.5
- new net N$14: R_ARRAY_2.4, R_ARRAY_2_CON.8
- new net N$15: R_ARRAY_2.5, R_ARRAY_2_CON.7
- new net N$16: R_ARRAY_2.6, R_ARRAY_2_CON.6
- new net N$17: R_ARRAY_2.7, R_ARRAY_2_CON.5
- new net N$18: R_ARRAY_2.8, R_ARRAY_2_CON.4
- new net N$19: R_ARRAY_2.9, R_ARRAY_2_CON.3
- new net N$2: LED1.C, R_ARRAY_1.9
- new net N$3: JP_DTA.1, U$1.D+, X1.D+
- new net N$4: JP_DTA.2, U$1.D-, X1.D-
- new net N$5: LED2.C, R_ARRAY_1.8
- new net N$6: LED3.C, R_ARRAY_1.7
- new net N$7: LED4.C, R_ARRAY_1.6
- new net N$8: LED1.A, LED_HEADER.1
- new net N$9: LED2.A, LED_HEADER.2
- new net R_ARRAY_1_8: BUTTON_1_SYNC.P1, R_ARRAY_1.2
- new net VCC: BUTTON_2.S, POWER.A, U$1.VBUS, VCC_RAIL_L.1, VCC_RAIL_L.10, VCC_RAIL_L.2, VCC_RAIL_L.3, VCC_RAIL_L.4, VCC_RAIL_L.5, VCC_RAIL_L.6, VCC_RAIL_L.7, VCC_RAIL_L.8, VCC_RAIL_L.9, VCC_RAIL_R.1, VCC_RAIL_R.10, VCC_RAIL_R.2, VCC_RAIL_R.3, VCC_RAIL_R.4, VCC_RAIL_R.5, VCC_RAIL_R.6, VCC_RAIL_R.7, VCC_RAIL_R.8, VCC_RAIL_R.9, X1.VBUS
- net GND: now also GND_RAIL_L.1, GND_RAIL_L.10, GND_RAIL_L.2, GND_RAIL_L.3, GND_RAIL_L.4, GND_RAIL_L.5, GND_RAIL_L.6, GND_RAIL_L.7, GND_RAIL_L.8, GND_RAIL_L.9, GND_RAIL_R.1, GND_RAIL_R.10, GND_RAIL_R.2, GND_RAIL_R.3, GND_RAIL_R.4, GND_RAIL_R.5, GND_RAIL_R.6, GND_RAIL_R.7, GND_RAIL_R.8, GND_RAIL_R.9, R_ARRAY_1.1, R_ARRAY_2.1, U$1.GND, X1.GND; no longer MCU_LEFT_SIDE.6, R_ARRAY_8.1
Other:
- moved on the sheet: POWER
