File: 2023/fDrive.RP2040/v1/BNSK-Rambo-Converters-Device.brd (EAGLE design)
At the start: 68 x 58 mm, 8 parts

Commit message: 2023.2. PCBs
Parts:
- added CHECKING: (no value), adafruit:1206
Connections:
- net MCU_D4: now also CHECKING.A
- net RA_6: now also CHECKING.C
Routing:
- net RA_1: track 77.7 -> 0.00 mm
- net GND: track 69.8 -> 0.00 mm
- net RA_2: track 58.5 -> 0.00 mm
- net MCU_D2: track 40.1 -> 0.00 mm
- net MCU_D3: track 36.6 -> 0.00 mm
- net RA_3: track 33.4 -> 0.00 mm
- net RA_5: track 31.3 -> 0.00 mm
- net MCU_D0: track 30.8 -> 0.00 mm
- net MCU_D1: track 23.5 -> 0.00 mm
- net RA_4: track 15.8 -> 0.00 mm
- net VCC_33: track 12.9 -> 0.00 mm
Other:
- board text added: "Converters Automation Device"
- board text added: "RAMBO"
- board text removed: "C:/DVT/Fred.PCB/2023/BNSK-Rambo-Converters-Device/Title.Converters Automation Device.bmp"
- board text removed: "C:/DVT/Fred.PCB/2023/BNSK-Rambo-Converters-Device/Title.fDrive.Logo.Gray.bmp"
- board text removed: "XIAO ESP32 C3"
