File: 2023/fDrive.RP2040/v1/fDrive.RP2040.sch (EAGLE design)
At the start: 8 parts

Commit message: 2023.2. PCBs
Parts:
- removed FAILED: (no value), adafruit:LEDSMT1206
- added AUTHORIZE: (no value), switch-omron:10-XX
- added BUTTON_PRESSED: (no value), adafruit:LEDSMT1206
- added FLASH_AT25SF321B_4MB: 25AA080SN, microchip:25AA080SN
- renumbered CHECK_NOW to MODE, PASSED to AUTHORIZED
Connections:
- removed net MCU_D10: MCU_LEFT_SIDE.4
- removed net MCU_D7: MCU_LEFT_SIDE.1
- removed net MCU_D8: MCU_LEFT_SIDE.2
- removed net MCU_D9: MCU_LEFT_SIDE.3
- removed net MCU_VCC_5V: MCU_LEFT_SIDE.7
- new net MCU_D10_MOSI: FLASH_AT25SF321B_4MB.SI, MCU_LEFT_SIDE.4
- new net MCU_D7_CS: FLASH_AT25SF321B_4MB.!CS, MCU_LEFT_SIDE.1
- new net MCU_D8_SCK: FLASH_AT25SF321B_4MB.SCK, MCU_LEFT_SIDE.2
- new net MCU_D9_MISO: FLASH_AT25SF321B_4MB.SO, MCU_LEFT_SIDE.3
- new net RA_7: BUTTON_PRESSED.C, R_ARRAY_8.8
- net GND: now also FLASH_AT25SF321B_4MB.GND
- net MCU_D1: now also RUNNING.A; no longer FAILED.A
- net MCU_D2: now also MODE.S; no longer RUNNING.A
- net MCU_D3: now also AUTHORIZE.S; no longer MODE.S
- net MCU_D4: now also BUTTON_PRESSED.A
- net RA_3: now also RUNNING.C; no longer FAILED.C
- net RA_4: no longer RUNNING.C
- net RA_6: now also AUTHORIZE.P1
- net VCC_33: now also FLASH_AT25SF321B_4MB.!HOLD, FLASH_AT25SF321B_4MB.!WP, FLASH_AT25SF321B_4MB.VCC
