File: 2023/NusbioV2.Board/bu/NusbioV2.Board.sch (EAGLE design)
At the start: 27 parts

Commit message: Nsubio /2 v2 update
Connections:
- net D0_SCLK: now also I2C_OUT_1.2, I2C_OUT_2.2; no longer I2C_OUT_1.1, I2C_OUT_2.1
- net D2_MISO: now also I2C_OUT_1.1, I2C_OUT_2.1; no longer I2C_OUT_1.2, I2C_OUT_2.2
Changed lines of the file:
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@@
-</segment>
-<segment>
-<pinref part="I2C_OUT_1" gate="A" pin="1"/>
-<wire x1="-121.92" y1="104.14" x2="-132.08" y2="104.14" width="0.1524" layer="91"/>
-<label x="-137.16" y="106.68" size="1.778" layer="95"/>
 </segment>
 <segment>
@@
 </segment>
 <segment>
-<pinref part="I2C_OUT_2" gate="A" pin="1"/>
-<wire x1="-121.92" y1="124.46" x2="-144.78" y2="124.46" width="0.1524" layer="91"/>
-<label x="-144.78" y="127" size="1.778" layer="95"/>
+<pinref part="I2C_OUT_2" gate="A" pin="2"/>
+<wire x1="-121.92" y1="121.92" x2="-144.78" y2="121.92" width="0.1524" layer="91"/>
+<label x="-142.24" y="121.92" size="1.778" layer="95"/>
+</segment>
+<segment>
+<pinref part="I2C_OUT_1" gate="A" pin="2"/>
+<wire x1="-121.92" y1="101.6" x2="-134.62" y2="101.6" width="0.1524" layer="91"/>
+<label x="-137.16" y="101.6" size="1.778" layer="95"/>
 </segment>
 </net>
@@
 </segment>
 <segment>
-<pinref part="I2C_OUT_1" gate="A" pin="2"/>
-<wire x1="-121.92" y1="101.6" x2="-134.62" y2="101.6" width="0.1524" layer="91"/>
-<label x="-137.16" y="101.6" size="1.778" layer="95"/>
-</segment>
-<segment>
-<pinref part="I2C_OUT_2" gate="A" pin="2"/>
-<wire x1="-121.92" y1="121.92" x2="-144.78" y2="121.92" width="0.1524" layer="91"/>
-<label x="-142.24" y="121.92" size="1.778" layer="95"/>
-</segment>
-<segment>
 <pinref part="I2C_DTA_CONN" gate="1" pin="O"/>
 <wire x1="-142.24" y1="40.64" x2="-160.02" y2="40.64" width="0.1524" layer="91"/>
 <label x="-162.56" y="43.18" size="1.778" layer="95"/>
 </segment>
+<segment>
+<pinref part="I2C_OUT_2" gate="A" pin="1"/>
+<wire x1="-121.92" y1="124.46" x2="-144.78" y2="124.46" width="0.1524" layer="91"/>
+<label x="-144.78" y="127" size="1.778" layer="95"/>
+</segment>
+<segment>
+<pinref part="I2C_OUT_1" gate="A" pin="1"/>
+<wire x1="-121.92" y1="104.14" x2="-132.08" y2="104.14" width="0.1524" layer="91"/>
+<label x="-137.16" y="106.68" size="1.778" layer="95"/>
+</segment>
 </net>
