File: 2023/NusbioV2.Board/bu/NusbioV2.Board.brd (EAGLE design)
At the start: 88 x 77 mm, 27 parts

Commit message: Fix Nusbio gnd pin for gpios led resitor array
Connections:
- net DO_NOT_USE: now also R_ARRAY_1.1; no longer R_ARRAY_1.10
- net GND: now also R_ARRAY_1.10; no longer R_ARRAY_1.1
Other:
- board text added: "PCBv3 - 2023.04"
- board text removed: "PCBv2 - 2023.03"
Changed lines of the file:
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@@
 <plain>
 <text x="46" y="73.5" size="3.81" layer="26" rot="SMR0" align="center">Nusbio /2</text>
-<text x="46" y="20.5" size="1.4224" layer="26" rot="MR0" align="center">PCBv2 - 2023.03</text>
+<text x="46" y="20.5" size="1.4224" layer="26" rot="MR0" align="center">PCBv3 - 2023.04</text>
 <text x="46" y="28.5" size="2.54" layer="26" rot="SMR0" align="center">www.FredericTorres.com</text>
 <text x="86.5" y="36" size="1.27" layer="25" rot="R270" align="center">GND</text>
@@
 <contactref element="SPI_OUT_1" pad="1"/>
 <contactref element="GPIO_OUT" pad="1"/>
-<contactref element="R_ARRAY_1" pad="1"/>
 <contactref element="SPI_OUT_2" pad="1"/>
 <contactref element="I2C_OUT_1" pad="4"/>
@@
 <contactref element="H3" pad="B3,3"/>
 <contactref element="H4" pad="B3,3"/>
+<contactref element="R_ARRAY_1" pad="10"/>
 <wire x1="81.62" y1="60" x2="84" y2="84" width="0" layer="19" extent="1-1"/>
 <wire x1="86.7" y1="40" x2="81.62" y2="60" width="0" layer="19" extent="1-1"/>
@@
 <wire x1="66.81" y1="15.7" x2="84" y2="19" width="0" layer="19" extent="1-1"/>
 <wire x1="45.63" y1="15.5" x2="66.81" y2="15.7" width="0" layer="19" extent="1-1"/>
-<wire x1="48.77" y1="88" x2="84" y2="84" width="0" layer="19" extent="1-1"/>
-<wire x1="23.89" y1="87.3" x2="48.77" y2="88" width="0" layer="19" extent="1-1"/>
-<wire x1="8" y1="84" x2="23.89" y2="87.3" width="0" layer="19" extent="1-1"/>
-<wire x1="12.152" y1="70" x2="8" y2="84" width="0" layer="19" extent="1-1"/>
-<wire x1="34.5" y1="63.585" x2="12.152" y2="70" width="0" layer="19" extent="1-1"/>
-<wire x1="4.5" y1="39.57" x2="12.152" y2="70" width="0" layer="19" extent="1-1"/>
+<wire x1="34.5" y1="40.725" x2="45.63" y2="15.5" width="0" layer="19" extent="1-1"/>
+<wire x1="4.5" y1="39.57" x2="34.5" y2="40.725" width="0" layer="19" extent="1-1"/>
 <wire x1="8" y1="19" x2="4.5" y2="39.57" width="0" layer="19" extent="1-1"/>
+<wire x1="12.152" y1="70" x2="4.5" y2="39.57" width="0" layer="19" extent="1-1"/>
+<wire x1="8" y1="84" x2="12.152" y2="70" width="0" layer="19" extent="1-1"/>
+<wire x1="23.89" y1="87.3" x2="8" y2="84" width="0" layer="19" extent="1-1"/>
+<wire x1="48.77" y1="88" x2="23.89" y2="87.3" width="0" layer="19" extent="1-1"/>
 </signal>
 <signal name="VCC_33">
@@
 <wire x1="22.77" y1="15.5" x2="23.5" y2="25.578" width="0" layer="19" extent="1-1"/>
 </signal>
-<signal name="DO_NOT_USE">
-<contactref element="R_ARRAY_1" pad="10"/>
-</signal>
 <signal name="R_G_0">
 <contactref element="R_ARRAY_1" pad="2"/>
@@
 <wire x1="27" y1="43.578" x2="27" y2="61.422" width="0" layer="19" extent="1-1"/>
 </signal>
+<signal name="DO_NOT_USE">
+<contactref element="R_ARRAY_1" pad="1"/>
+</signal>
 </signals>

Commit message: Nusbio /2 v3
Parts:
- added LED_I2C_MODE: (no value), adafruit:1206
- added R_LED_I2C_MODE: (no value), adafruit:R1206
Connections:
- new net N$3: LED_I2C_MODE.C, R_LED_I2C_MODE.2
- net D1_MOSI: now also I2C_OUT_1.1, I2C_OUT_2.1
- net D2_MISO: no longer I2C_OUT_1.1, I2C_OUT_2.1
- net GND: now also R_LED_I2C_MODE.1
- net N$2: now also LED_I2C_MODE.A
