File: 2023/Nusbio Test GPIOS Extension/bu/Nusbio Test GPIOS Extension.brd (EAGLE design)
At the start: 44 x 50 mm, 7 parts

Commit message: Nusbio /2 v3
Parts:
- removed SOIC8_208MIL_EEPROM: (no value), microbuilder:SOIC8_208MIL
- added SPI_SOIC_8_FLASH: 25AA080SN, microchip:SO-08
- moved USE_CS_3 3.81 mm to (38.0, 13.0)
- moved USE_CS_4 3.81 mm to (38.0, 20.0)
Connections:
- net CS: now also SPI_SOIC_8_FLASH.1; no longer SOIC8_208MIL_EEPROM.1
- net GND: now also SPI_SOIC_8_FLASH.4; no longer SOIC8_208MIL_EEPROM.4
- net MISO: now also SPI_SOIC_8_FLASH.2; no longer SOIC8_208MIL_EEPROM.2
- net MOSI: now also SPI_SOIC_8_FLASH.5; no longer SOIC8_208MIL_EEPROM.5
- net SCK: now also SPI_SOIC_8_FLASH.6; no longer SOIC8_208MIL_EEPROM.6
- net VCC: now also SPI_SOIC_8_FLASH.3, SPI_SOIC_8_FLASH.7, SPI_SOIC_8_FLASH.8; no longer SOIC8_208MIL_EEPROM.3, SOIC8_208MIL_EEPROM.7, SOIC8_208MIL_EEPROM.8
Changed lines of the file:
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@@
 <attribute name="NAME" x="38.33" y="47.79" size="0.8128" layer="25" ratio="10" align="center"/>
+</element>
+<element name="SPI_SOIC_8_FLASH" library="microchip" package="SO-08" value="25AA080SN" x="21.5" y="20" smashed="yes" rot="R270">
+<attribute name="MF" value="MICROCHIP" x="21.5" y="20" size="1.778" layer="27" rot="R270" display="off"/>
+<attribute name="MPN" value="25AA080/SN" x="21.5" y="20" size="1.778" layer="27" rot="R270" display="off"/>
+<attribute name="NAME" x="13.095" y="26" size="1.27" layer="25"/>
+<attribute name="OC_FARNELL" value="1816072" x="21.5" y="20" size="1.778" layer="27" rot="R270" display="off"/>
+<attribute name="OC_NEWARK" value="92C7351" x="21.5" y="20" size="1.778" layer="27" rot="R270" display="off"/>
 </element>
 <element name="R_4K" library="adafruit" package="R1206" value="" x="6.5" y="24.5" smashed="yes" rot="R180">
@@
 <attribute name="VALUE" x="7.659" y="19.3495" size="1.27" layer="27" rot="R180"/>
 </element>
-<element name="USE_CS_3" library="microbuilder" package="SOLDERJUMPER_REFLOW" value="" x="36.5" y="16.5" smashed="yes">
-<attribute name="NAME" x="36.849" y="18.5" size="0.8128" layer="25" ratio="18" align="center"/>
-<attribute name="VALUE" x="36.9001" y="16.5" size="0.02" layer="27"/>
+<element name="USE_CS_3" library="microbuilder" package="SOLDERJUMPER_REFLOW" value="" x="38" y="13" smashed="yes">
+<attribute name="NAME" x="38.349" y="15" size="0.8128" layer="25" ratio="18" align="center"/>
+<attribute name="VALUE" x="38.4001" y="13" size="0.02" layer="27"/>
 </element>
-<element name="USE_CS_4" library="microbuilder" package="SOLDERJUMPER_REFLOW" value="" x="36.5" y="23.5" smashed="yes">
-<attribute name="NAME" x="36.849" y="25.5" size="0.8128" layer="25" ratio="18" align="center"/>
-<attribute name="VALUE" x="36.9001" y="23.5" size="0.02" layer="27"/>
-</element>
-<element name="SOIC8_208MIL_EEPROM" library="microbuilder" package="SOIC8_208MIL" value="" x="21.5" y="20" smashed="yes" rot="R270">
-<attribute name="NAME" x="21.635" y="24.405" size="0.8128" layer="25" ratio="18" align="center"/>
-<attribute name="VALUE" x="21.119" y="21.905" size="0.4064" layer="27" ratio="10" rot="R270"/>
+<element name="USE_CS_4" library="microbuilder" package="SOLDERJUMPER_REFLOW" value="" x="38" y="20" smashed="yes">
+<attribute name="NAME" x="38.349" y="22" size="0.8128" layer="25" ratio="18" align="center"/>
+<attribute name="VALUE" x="38.4001" y="20" size="0.02" layer="27"/>
 </element>
 </elements>
@@
 <contactref element="GPIO_IN" pad="10"/>
 <contactref element="GPIO_OUT" pad="10"/>
+<contactref element="SPI_SOIC_8_FLASH" pad="4"/>
 <contactref element="R_4K" pad="1"/>
-<contactref element="SOIC8_208MIL_EEPROM" pad="4"/>
-<wire x1="18.185" y1="18.095" x2="33.43" y2="48" width="0" layer="19" extent="1-1"/>
-<wire x1="7.922" y1="24.5" x2="18.185" y2="18.095" width="0" layer="19" extent="1-1"/>
-<wire x1="10.922071875" y1="2.37569375" x2="18.185" y2="18.095" width="0" layer="19" extent="1-1"/>
+<wire x1="18.9" y1="18.095" x2="33.43" y2="48" width="0" layer="19" extent="1-1"/>
+<wire x1="7.922" y1="24.5" x2="18.9" y2="18.095" width="0" layer="19" extent="1-1"/>
+<wire x1="10.922071875" y1="2.37569375" x2="18.9" y2="18.095" width="0" layer="19" extent="1-1"/>
 </signal>
 <signal name="VCC">
 <contactref element="GPIO_IN" pad="9"/>
 <contactref element="GPIO_OUT" pad="9"/>
+<contactref element="SPI_SOIC_8_FLASH" pad="8"/>
+<contactref element="SPI_SOIC_8_FLASH" pad="7"/>
 <contactref element="LED_POWER" pad="A"/>
-<contactref element="SOIC8_208MIL_EEPROM" pad="8"/>
-<contactref element="SOIC8_208MIL_EEPROM" pad="3"/>
-<contactref element="SOIC8_208MIL_EEPROM" pad="7"/>
-<wire x1="24.815" y1="21.905" x2="30.89" y2="48" width="0" layer="19" extent="1-1"/>
-<wire x1="24.815" y1="20.635" x2="24.815" y2="21.905" width="0" layer="19" extent="1-1"/>
-<wire x1="18.185" y1="19.365" x2="24.815" y2="20.635" width="0" layer="19" extent="1-1"/>
-<wire x1="7.811" y1="16.8095" x2="18.185" y2="19.365" width="0" layer="19" extent="1-1"/>
+<contactref element="SPI_SOIC_8_FLASH" pad="3"/>
+<wire x1="24.1" y1="21.905" x2="30.89" y2="48" width="0" layer="19" extent="1-1"/>
+<wire x1="24.1" y1="20.635" x2="24.1" y2="21.905" width="0" layer="19" extent="1-1"/>
+<wire x1="18.9" y1="19.365" x2="24.1" y2="20.635" width="0" layer="19" extent="1-1"/>
+<wire x1="7.811" y1="16.8095" x2="18.9" y2="19.365" width="0" layer="19" extent="1-1"/>
 <wire x1="13.462071875" y1="2.37569375" x2="7.811" y2="16.8095" width="0" layer="19" extent="1-1"/>
 </signal>
 <signal name="SCK">
 <contactref element="GPIO_IN" pad="1"/>
+<contactref element="SPI_SOIC_8_FLASH" pad="6"/>
 <contactref element="GPIO_OUT" pad="1"/>
-<contactref element="SOIC8_208MIL_EEPROM" pad="6"/>
-<wire x1="24.815" y1="19.365" x2="10.57" y2="48" width="0" layer="19" extent="1-1"/>
-<wire x1="33.782071875" y1="2.37569375" x2="24.815" y2="19.365" width="0" layer="19" extent="1-1"/>
+<wire x1="24.1" y1="19.365" x2="10.57" y2="48" width="0" layer="19" extent="1-1"/>
+<wire x1="33.782071875" y1="2.37569375" x2="24.1" y2="19.365" width="0" layer="19" extent="1-1"/>
 </signal>
 <signal name="MOSI">
 <contactref element="GPIO_IN" pad="2"/>
+<contactref element="SPI_SOIC_8_FLASH" pad="5"/>
 <contactref element="GPIO_OUT" pad="2"/>
-<contactref element="SOIC8_208MIL_EEPROM" pad="5"/>
-<wire x1="24.815" y1="18.095" x2="13.11" y2="48" width="0" layer="19" extent="1-1"/>
-<wire x1="31.242071875" y1="2.37569375" x2="24.815" y2="18.095" width="0" layer="19" extent="1-1"/>
+<wire x1="24.1" y1="18.095" x2="13.11" y2="48" width="0" layer="19" extent="1-1"/>
+<wire x1="31.242071875" y1="2.37569375" x2="24.1" y2="18.095" width="0" layer="19" extent="1-1"/>
 </signal>
 <signal name="MISO">
 <contactref element="GPIO_IN" pad="3"/>
+<contactref element="SPI_SOIC_8_FLASH" pad="2"/>
 <contactref element="GPIO_OUT" pad="3"/>
-<contactref element="SOIC8_208MIL_EEPROM" pad="2"/>
-<wire x1="18.185" y1="20.635" x2="15.65" y2="48" width="0" layer="19" extent="1-1"/>
-<wire x1="28.702071875" y1="2.37569375" x2="18.185" y2="20.635" width="0" layer="19" extent="1-1"/>
+<wire x1="18.9" y1="20.635" x2="15.65" y2="48" width="0" layer="19" extent="1-1"/>
+<wire x1="28.702071875" y1="2.37569375" x2="18.9" y2="20.635" width="0" layer="19" extent="1-1"/>
 </signal>
 <signal name="CS">
+<contactref element="SPI_SOIC_8_FLASH" pad="1"/>
 <contactref element="USE_CS_3" pad="2"/>
 <contactref element="USE_CS_4" pad="2"/>
-<contactref element="SOIC8_208MIL_EEPROM" pad="1"/>
-<wire x1="37.262" y1="16.5" x2="37.262" y2="23.5" width="0" layer="19" extent="1-1"/>
-<wire x1="18.185" y1="21.905" x2="37.262" y2="23.5" width="0" layer="19" extent="1-1"/>
+<wire x1="38.762" y1="13" x2="38.762" y2="20" width="0" layer="19" extent="1-1"/>
+<wire x1="18.9" y1="21.905" x2="38.762" y2="20" width="0" layer="19" extent="1-1"/>
 </signal>
 <signal name="GPIO6">
@@
 <contactref element="GPIO_OUT" pad="5"/>
 <contactref element="USE_CS_4" pad="1"/>
-<wire x1="35.738" y1="23.5" x2="20.73" y2="48" width="0" layer="19" extent="1-1"/>
-<wire x1="23.622071875" y1="2.37569375" x2="35.738" y2="23.5" width="0" layer="19" extent="1-1"/>
+<wire x1="37.238" y1="20" x2="20.73" y2="48" width="0" layer="19" extent="1-1"/>
+<wire x1="23.622071875" y1="2.37569375" x2="37.238" y2="20" width="0" layer="19" extent="1-1"/>
 </signal>
 <signal name="CS_3">
@@
 <contactref element="GPIO_OUT" pad="4"/>
 <contactref element="USE_CS_3" pad="1"/>
-<wire x1="35.738" y1="16.5" x2="18.19" y2="48" width="0" layer="19" extent="1-1"/>
-<wire x1="26.162071875" y1="2.37569375" x2="35.738" y2="16.5" width="0" layer="19" extent="1-1"/>
+<wire x1="37.238" y1="13" x2="18.19" y2="48" width="0" layer="19" extent="1-1"/>
+<wire x1="26.162071875" y1="2.37569375" x2="37.238" y2="13" width="0" layer="19" extent="1-1"/>
 </signal>
 </signals>
