File: 2023/Nusbio SPI Extension/Nusbio SPI Extension.sch (EAGLE design)
At the start: 9 parts

Commit message: Nusbio v2 pcb and SPIExtension v 1 2023/05
Parts:
- added H1, H2, H3: MOUNT-PAD-ROUND2.8, holes:MOUNT-PAD-ROUND2.8
Changed lines of the file:
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@@
 <part name="GND7" library="supply1" deviceset="GND" device=""/>
 <part name="GND8" library="supply1" deviceset="GND" device=""/>
+<part name="H2" library="holes" library_urn="urn:adsk.eagle:library:237" deviceset="MOUNT-PAD-ROUND" device="2.8" package3d_urn="urn:adsk.eagle:package:14281/1"/>
+<part name="H1" library="holes" library_urn="urn:adsk.eagle:library:237" deviceset="MOUNT-PAD-ROUND" device="2.8" package3d_urn="urn:adsk.eagle:package:14281/1"/>
+<part name="H3" library="holes" library_urn="urn:adsk.eagle:library:237" deviceset="MOUNT-PAD-ROUND" device="2.8" package3d_urn="urn:adsk.eagle:package:14281/1"/>
 </parts>
 <sheets>
@@
 <attribute name="VALUE" x="121.92" y="111.76" size="1.778" layer="96" rot="R90"/>
 </instance>
+<instance part="H2" gate="G$1" x="-66.04" y="154.94" smashed="yes">
+<attribute name="NAME" x="-63.246" y="155.5242" size="1.778" layer="95"/>
+<attribute name="VALUE" x="-63.246" y="152.4762" size="1.778" layer="96"/>
+</instance>
+<instance part="H1" gate="G$1" x="-63.5" y="165.1" smashed="yes">
+<attribute name="NAME" x="-60.706" y="165.6842" size="1.778" layer="95"/>
+<attribute name="VALUE" x="-60.706" y="162.6362" size="1.778" layer="96"/>
+</instance>
+<instance part="H3" gate="G$1" x="-20.32" y="154.94" smashed="yes">
+<attribute name="NAME" x="-17.526" y="155.5242" size="1.778" layer="95"/>
+<attribute name="VALUE" x="-17.526" y="152.4762" size="1.778" layer="96"/>
+</instance>
 </instances>
 <busses>
@@
 </schematic>
 </drawing>
+<compatibility>
+<note version="8.2" severity="warning">
+Since Version 8.2, EAGLE supports online libraries. The ids
+of those online libraries will not be understood (or retained)
+with this version.
+</note>
+<note version="8.3" severity="warning">
+Since Version 8.3, EAGLE supports URNs for individual library
+assets (packages, symbols, and devices). The URNs of those assets
+will not be understood (or retained) with this version.
+</note>
+<note version="8.3" severity="warning">
+Since Version 8.3, EAGLE supports the association of 3D packages
+with devices in libraries, schematics, and board files. Those 3D
+packages will not be understood (or retained) with this version.
+</note>
+</compatibility>
 </eagle>
