File: 2023/French USB C/French USB C.brd (EAGLE design)
At the start: 30 x 45 mm, 6 parts, among them X1 USB-A

Commit message: usb multiplicator 2023 / French USBC
Connections:
- net N$1 renamed GND_W
- net N$3 renamed D_PLUS
- net N$4 renamed D_MINUS
Routing:
- net GND_W: track 69.4 -> 0.00 mm
- net VCC: track 38.0 -> 0.00 mm
- net D_MINUS: track 37.1 -> 0.00 mm
- net D_PLUS: track 35.8 -> 0.00 mm
- net N$5: track 10.9 -> 0.00 mm
- net N$2: track 10.2 -> 0.00 mm
- net N$6: track 10.1 -> 0.00 mm
Other:
- board text added: "PCBv2 - 2019.09"
- board text removed: "PCBv3 - 2023.03"
Changed lines of the file:
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@@
 <wire x1="0" y1="45" x2="0" y2="41" width="0" layer="20"/>
 <text x="12.5195" y="8.286" size="1.016" layer="25" rot="R180">GND</text>
-<text x="28.3365" y="23.0595" size="1.778" layer="26" rot="MR270" align="center">PCBv3 - 2023.03</text>
-<text x="3.935" y="22.887" size="2.54" layer="26" rot="MR270" align="center">FredericTorres.com</text>
+<text x="3" y="55" size="1.778" layer="26" rot="MR270" align="center">PCBv2 - 2019.09</text>
+<text x="16" y="38" size="3.81" layer="26" rot="MR270" align="center">FredericTorres.com</text>
 <text x="25.9" y="7" size="1.016" layer="25" rot="R180">GND</text>
 <wire x1="0" y1="4" x2="0" y2="0" width="0" layer="20"/>
@@
 <autorouter>
 <pass name="Default">
-<param name="RoutingGrid" value="4.92125984mil"/>
+<param name="RoutingGrid" value="0.125mm"/>
 <param name="AutoGrid" value="1"/>
 <param name="Efforts" value="1"/>
@@
 </elements>
 <signals>
-<signal name="N$1">
+<signal name="GND_W">
 <contactref element="X1" pad="4"/>
 <contactref element="U$1" pad="GND"/>
 <contactref element="RN1" pad="1"/>
-<wire x1="10.9728" y1="39.0906" x2="10.9728" y2="5.2578" width="0.254" layer="1"/>
-<wire x1="10.9728" y1="5.2578" x2="11" y2="5.1" width="0.254" layer="1"/>
-<wire x1="10.9728" y1="39.0906" x2="10.9" y2="39.2" width="0.254" layer="1"/>
-<wire x1="25.3746" y1="10.5156" x2="25.3746" y2="10.0584" width="0.254" layer="16"/>
-<wire x1="14.4018" y1="21.4884" x2="25.3746" y2="10.5156" width="0.254" layer="16"/>
-<wire x1="14.4018" y1="35.6616" x2="14.4018" y2="21.4884" width="0.254" layer="16"/>
-<wire x1="10.9728" y1="39.0906" x2="14.4018" y2="35.6616" width="0.254" layer="16"/>
-<wire x1="25.3746" y1="10.0584" x2="25.5" y2="10.04" width="0.254" layer="16"/>
-<wire x1="10.9728" y1="39.0906" x2="10.9" y2="39.2" width="0.254" layer="16"/>
+<wire x1="25.5" y1="10.04" x2="10.9" y2="39.2" width="0" layer="19" extent="1-1"/>
+<wire x1="11" y1="5.1" x2="25.5" y2="10.04" width="0" layer="19" extent="1-1"/>
 </signal>
-<signal name="N$3">
+<signal name="D_PLUS">
 <contactref element="X1" pad="3"/>
 <contactref element="U$1" pad="D+"/>
-<wire x1="13.4874" y1="10.7442" x2="13.4874" y2="5.2578" width="0.254" layer="1"/>
-<wire x1="11.43" y1="12.8016" x2="13.4874" y2="10.7442" width="0.254" layer="1"/>
-<wire x1="11.43" y1="37.2618" x2="11.43" y2="12.8016" width="0.254" layer="1"/>
-<wire x1="13.2588" y1="39.0906" x2="11.43" y2="37.2618" width="0.254" layer="1"/>
-<wire x1="13.4874" y1="5.2578" x2="13.5" y2="5.1" width="0.254" layer="1"/>
-<wire x1="13.2588" y1="39.0906" x2="13.4" y2="39.2" width="0.254" layer="1"/>
+<wire x1="13.5" y1="5.1" x2="13.4" y2="39.2" width="0" layer="19" extent="1-1"/>
 </signal>
-<signal name="N$4">
+<signal name="D_MINUS">
 <contactref element="X1" pad="2"/>
 <contactref element="U$1" pad="D-"/>
-<wire x1="15.3162" y1="9.6012" x2="15.3162" y2="5.2578" width="0.254" layer="1"/>
-<wire x1="11.8872" y1="13.0302" x2="15.3162" y2="9.6012" width="0.254" layer="1"/>
-<wire x1="11.8872" y1="35.6616" x2="11.8872" y2="13.0302" width="0.254" layer="1"/>
-<wire x1="15.3162" y1="39.0906" x2="11.8872" y2="35.6616" width="0.254" layer="1"/>
-<wire x1="15.3162" y1="5.2578" x2="15.5" y2="5.1" width="0.254" layer="1"/>
-<wire x1="15.3162" y1="39.0906" x2="15.4" y2="39.2" width="0.254" layer="1"/>
+<wire x1="15.5" y1="5.1" x2="15.4" y2="39.2" width="0" layer="19" extent="1-1"/>
 </signal>
 <signal name="VCC">
@@
 <contactref element="L_WHITE" pad="A"/>
 <contactref element="L_RED" pad="A"/>
-<wire x1="17.8308" y1="8.9154" x2="17.8308" y2="5.2578" width="0.254" layer="1"/>
-<wire x1="13.2588" y1="13.4874" x2="17.8308" y2="8.9154" width="0.254" layer="1"/>
-<wire x1="17.8308" y1="5.2578" x2="18" y2="5.1" width="0.254" layer="1"/>
-<wire x1="13.2588" y1="13.4874" x2="13.23" y2="13.5" width="0.254" layer="1"/>
-<wire x1="17.8308" y1="35.2044" x2="17.8308" y2="39.0906" width="0.254" layer="1"/>
-<wire x1="13.2588" y1="30.6324" x2="17.8308" y2="35.2044" width="0.254" layer="1"/>
-<wire x1="17.8308" y1="39.0906" x2="17.9" y2="39.2" width="0.254" layer="1"/>
-<wire x1="13.2588" y1="30.6324" x2="13.23" y2="30.5" width="0.254" layer="1"/>
-<wire x1="13.2588" y1="30.4038" x2="13.2588" y2="22.1742" width="0.254" layer="1"/>
-<wire x1="13.2588" y1="22.1742" x2="13.23" y2="22" width="0.254" layer="1"/>
-<wire x1="13.2588" y1="30.4038" x2="13.23" y2="30.5" width="0.254" layer="1"/>
-<wire x1="13.2588" y1="21.9456" x2="13.2588" y2="13.716" width="0.254" layer="1"/>
-<wire x1="13.2588" y1="13.716" x2="13.23" y2="13.5" width="0.254" layer="1"/>
-<wire x1="13.2588" y1="21.9456" x2="13.23" y2="22" width="0.254" layer="1"/>
+<wire x1="13.23" y1="30.5" x2="17.9" y2="39.2" width="0" layer="19" extent="1-1"/>
+<wire x1="13.23" y1="22" x2="13.23" y2="30.5" width="0" layer="19" extent="1-1"/>
+<wire x1="13.23" y1="13.5" x2="13.23" y2="22" width="0" layer="19" extent="1-1"/>
+<wire x1="18" y1="5.1" x2="13.23" y2="13.5" width="0" layer="19" extent="1-1"/>
 </signal>
 <signal name="N$2">
 <contactref element="L_BLUE" pad="K"/>
 <contactref element="RN1" pad="2"/>
-<wire x1="16.4592" y1="12.8016" x2="25.3746" y2="12.8016" width="0.254" layer="1"/>
-<wire x1="15.7734" y1="13.4874" x2="16.4592" y2="12.8016" width="0.254" layer="1"/>
-<wire x1="25.3746" y1="12.8016" x2="25.5" y2="12.58" width="0.254" layer="1"/>
-<wire x1="15.7734" y1="13.4874" x2="15.77" y2="13.5" width="0.254" layer="1"/>
+<wire x1="15.77" y1="13.5" x2="25.5" y2="12.58" width="0" layer="19" extent="1-1"/>
 </signal>
 <signal name="N$6">
 <contactref element="L_WHITE" pad="K"/>
 <contactref element="RN1" pad="6"/>
-<wire x1="16.2306" y1="22.6314" x2="25.3746" y2="22.6314" width="0.254" layer="1"/>
-<wire x1="15.7734" y1="22.1742" x2="16.2306" y2="22.6314" width="0.254" layer="1"/>
-<wire x1="25.3746" y1="22.6314" x2="25.5" y2="22.74" width="0.254" layer="1"/>
-<wire x1="15.7734" y1="22.1742" x2="15.77" y2="22" width="0.254" layer="1"/>
+<wire x1="15.77" y1="22" x2="25.5" y2="22.74" width="0" layer="19" extent="1-1"/>
 </signal>
 <signal name="N$5">
 <contactref element="L_RED" pad="K"/>
 <contactref element="RN1" pad="8"/>
-<wire x1="18.288" y1="27.8892" x2="25.3746" y2="27.8892" width="0.254" layer="1"/>
-<wire x1="15.7734" y1="30.4038" x2="18.288" y2="27.8892" width="0.254" layer="1"/>
-<wire x1="25.3746" y1="27.8892" x2="25.5" y2="27.82" width="0.254" layer="1"/>
-<wire x1="15.7734" y1="30.4038" x2="15.77" y2="30.5" width="0.254" layer="1"/>
+<wire x1="15.77" y1="30.5" x2="25.5" y2="27.82" width="0" layer="19" extent="1-1"/>
 </signal>
 </signals>
