File: 2023/UpTo11.2023/MotherBoard/UpTo11.MotherBoard.sch (EAGLE design)
At the start: 9 parts, among them X1 USB-A

Commit message: Upto11 2023
Parts:
- removed 2N3904_NPN: 2N3904, transistor:2N3904
- removed 2N3906_PNP: 2N3906, transistor-pnp:2N3906
- removed R_100_O, R_1M_O, R_22_O, R_PWR_LED_1K: (no value), adafruit:R-US_0207/10
- added H1, H2, H3, H4: MOUNT-PAD-ROUND3.3, holes:MOUNT-PAD-ROUND3.3
- added POWER: (no value), adafruit:LEDSMT1206
- added R_1K: (no value), adafruit:R-US_R1206
Connections:
- removed net LED_FLASH: 2N3904_NPN.E, FRONT_PANEL_INTERFACE.4
- removed net LED_PWR: FRONT_PANEL_INTERFACE.3, R_PWR_LED_1K.1
- removed net N$2: 2N3904_NPN.C, CAP_100UF.2, R_22_O.1
- removed net N$5: 2N3906_PNP.B, CAP_100UF.1, R_1M_O.2
- removed net N$6: 2N3906_PNP.C, R_100_O.1
- removed net POT_IN: FRONT_PANEL_INTERFACE.5, R_100_O.2
- removed net POT_OUT: 2N3904_NPN.B, FRONT_PANEL_INTERFACE.6
- new net VCC_1K: CAP_100UF.2, FRONT_PANEL_INTERFACE.3, R_1K.1
- net GND_EX: now also CAP_100UF.1, POWER.C; no longer R_1M_O.1
- net VCC: now also POWER.A, R_1K.2; no longer 2N3906_PNP.E, R_22_O.2, R_PWR_LED_1K.2

Commit message: Upto11 2023
Parts:
- renumbered POWER to CONNECTED
Connections:
- net VCC: no longer CONNECTED.A
- net VCC_1K: now also CONNECTED.A
Changed lines of the file:
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@@
 <part name="H3" library="holes" library_urn="urn:adsk.eagle:library:237" deviceset="MOUNT-PAD-ROUND" device="3.3" package3d_urn="urn:adsk.eagle:package:14283/1"/>
 <part name="H4" library="holes" library_urn="urn:adsk.eagle:library:237" deviceset="MOUNT-PAD-ROUND" device="3.3" package3d_urn="urn:adsk.eagle:package:14283/1"/>
-<part name="POWER" library="adafruit" deviceset="LED" device="SMT1206"/>
+<part name="CONNECTED" library="adafruit" deviceset="LED" device="SMT1206"/>
 <part name="R_1K" library="adafruit" deviceset="R-US_" device="R1206"/>
 </parts>
@@
 <attribute name="VALUE" x="109.474" y="109.2962" size="1.778" layer="96"/>
 </instance>
-<instance part="POWER" gate="G$1" x="53.34" y="63.5" smashed="yes">
+<instance part="CONNECTED" gate="G$1" x="53.34" y="63.5" smashed="yes">
 <attribute name="NAME" x="56.896" y="58.928" size="1.778" layer="95" rot="R90"/>
 <attribute name="VALUE" x="59.055" y="58.928" size="1.778" layer="96" rot="R90"/>
@@
 </segment>
 <segment>
-<pinref part="POWER" gate="G$1" pin="C"/>
+<pinref part="CONNECTED" gate="G$1" pin="C"/>
 <wire x1="53.34" y1="58.42" x2="53.34" y2="48.26" width="0.1524" layer="91"/>
 <label x="60.96" y="50.8" size="1.778" layer="95"/>
@@
 <wire x1="86.36" y1="86.36" x2="86.36" y2="101.6" width="0.1524" layer="91"/>
 <label x="78.74" y="91.44" size="1.778" layer="95"/>
-</segment>
-<segment>
-<pinref part="POWER" gate="G$1" pin="A"/>
-<wire x1="53.34" y1="66.04" x2="53.34" y2="76.2" width="0.1524" layer="91"/>
-<label x="58.42" y="71.12" size="1.778" layer="95"/>
 </segment>
 <segment>
@@
 <label x="111.76" y="33.02" size="1.778" layer="95"/>
 </segment>
+<segment>
+<pinref part="CONNECTED" gate="G$1" pin="A"/>
+<wire x1="53.34" y1="66.04" x2="53.34" y2="76.2" width="0.1524" layer="91"/>
+<label x="58.42" y="71.12" size="1.778" layer="95"/>
+</segment>
 </net>
