File: 2023/UpTo11.2023/MotherBoard/UpTo11.MotherBoard.brd (EAGLE design)
At the start: 88 x 78 mm, 9 parts, among them X1 USB-A

Commit message: Upto11 2023
Parts:
- moved X1 55.0 mm to (87.0, 50.3), turned to 90 degrees
- renumbered POWER to CONNECTED
Connections:
- net VCC: no longer CONNECTED.A
- net VCC_1K: now also CONNECTED.A
Routing:
- net VCC: track 1.35 -> 135.0 mm
- net VCC_1K: track 0.00 -> 91.4 mm
- net GND_EX: track 0.11 -> 87.8 mm
Other:
- board text removed: "C:/DVT/Fred.PCB/2023/UpTo11.2023/FrontPanel/Title1.bmp"

Commit message: BNSK Booster v 2
Parts:
- added CN1: (no value), microbuilder:USB_HOST-PTH
- moved CONNECTED 34.0 mm to (44.0, 31.0), turned to 180 degrees
- moved R_1K 20.5 mm to (43.9, 39.0)
- moved CAP_100UF 9.06 mm to (45.0, 59.0)
- moved FRONT_PANEL_INTERFACE 2.00 mm to (46.0, 87.5)
- moved X1 0.30 mm to (87.0, 50.0)
Connections:
- removed net VCC_1K: CAP_100UF.2, CONNECTED.A, FRONT_PANEL_INTERFACE.3, R_1K.1
- new net DMINUS: CN1.D+, X1.2
- new net DPLUS: CN1.D-, X1.3
- new net N$1: CONNECTED.A, R_1K.1
- net GND_EX: now also CN1.GND
- net VCC: now also CAP_100UF.2, CN1.VBUS, FRONT_PANEL_INTERFACE.6; no longer FRONT_PANEL_INTERFACE.2
Routing:
- net VCC: track 135.0 -> 0.00 mm
- net VCC_1K: track 91.4 -> 0.00 mm
- net GND_EX: track 87.8 -> 0.11 mm
Other:
- board text added: "BNSK Booster - Mother Board"
- board text removed: "Cloud Booster- Mother Board"
- board text removed: "VCC_1K"
