File: 2023/UpTo11.2023/FrontPanel/v1/UpTo11.FrontPanel.sch (EAGLE design)
At the start: 6 parts, among them X1 USB-A

Commit message: BNSK Booster v 2
Parts:
- removed L_BLUE, L_RED, L_WHITE: (no value), adafruit:LED5MM
- removed RN1: (no value), resistor-sip:4610X
- removed U$1: USB, STUNTAZ:USB
- removed X1: USB-A, adafruit:USB-A
- added BOOSTER_ON_LED, DIAL_LED: (no value), adafruit:LED5MM
- added CONNECTED: (no value), adafruit:LEDSMT1206
- added FRONT_PANEL_INTERFACE: (no value), adafruit:PINHD-1X6
- added H1, H2, H3, H4: MOUNT-PAD-ROUND3.3, holes:MOUNT-PAD-ROUND3.3
- added POT_GND_(LEFT), POT_IN_(RIGHT), POT_OUT_(MIDDLE), SWITCH_IN, SWITCH_OUT: (no value), microbuilder:SOLDERJUMPERREFLOW
Connections:
- removed net N$1: RN1.1, U$1.GND, X1.GND
- removed net N$2: L_BLUE.C, RN1.2
- removed net N$3: U$1.D+, X1.D+
- removed net N$4: U$1.D-, X1.D-
- removed net N$5: L_RED.C, RN1.8
- removed net N$6: L_WHITE.C, RN1.6
- new net BOOSTER_ON: BOOSTER_ON_LED.A, POT_IN_(RIGHT).2, SWITCH_OUT.2
- new net DIAL_INPUT: DIAL_LED.A, POT_OUT_(MIDDLE).2
- new net GND_EX: BOOSTER_ON_LED.C, CONNECTED.C, DIAL_LED.C, FRONT_PANEL_INTERFACE.1, POT_GND_(LEFT).2
- new net VCC_1K: CONNECTED.A, FRONT_PANEL_INTERFACE.3, SWITCH_IN.2
- net VCC: now also FRONT_PANEL_INTERFACE.2; no longer L_BLUE.A, L_RED.A, L_WHITE.A, U$1.VBUS, X1.VBUS
