File: 2023/UpTo11.2023/MotherBoard/v1/UpTo11.MotherBoard.sch (EAGLE design)
At the start: 10 parts, among them X1 USB-A

Commit message: BNSK Booster v 2
Parts:
- removed CN1: (no value), microbuilder:USB_TYPEAPTHFML
Connections:
- removed net DMINUS: CN1.D+, X1.D-
- removed net DPLUS: CN1.D-, X1.D+
- removed net N$1: CONNECTED.A, R_1K.1
- new net VCC_1K: CAP_100UF.2, CONNECTED.A, FRONT_PANEL_INTERFACE.3, R_1K.1
- net GND_EX: no longer CN1.GND
- net VCC: now also FRONT_PANEL_INTERFACE.2; no longer CAP_100UF.2, CN1.VBUS, FRONT_PANEL_INTERFACE.6
Other:
- moved on the sheet: CONNECTED, R_1K
Changed lines of the file:
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@@
 <part name="CONNECTED" library="adafruit" deviceset="LED" device="SMT1206"/>
 <part name="R_1K" library="adafruit" deviceset="R-US_" device="R1206"/>
-<part name="CN1" library="microbuilder" deviceset="USB_TYPEA" device="PTHFML"/>
 </parts>
 <sheets>
@@
 <attribute name="VALUE" x="109.474" y="109.2962" size="1.778" layer="96"/>
 </instance>
-<instance part="CONNECTED" gate="G$1" x="43.18" y="50.8" smashed="yes">
-<attribute name="NAME" x="46.736" y="46.228" size="1.778" layer="95" rot="R90"/>
-<attribute name="VALUE" x="48.895" y="46.228" size="1.778" layer="96" rot="R90"/>
+<instance part="CONNECTED" gate="G$1" x="53.34" y="63.5" smashed="yes">
+<attribute name="NAME" x="56.896" y="58.928" size="1.778" layer="95" rot="R90"/>
+<attribute name="VALUE" x="59.055" y="58.928" size="1.778" layer="96" rot="R90"/>
 </instance>
-<instance part="R_1K" gate="G$1" x="43.18" y="63.5" smashed="yes" rot="R90">
-<attribute name="NAME" x="41.6814" y="59.69" size="1.778" layer="95" rot="R90"/>
-<attribute name="VALUE" x="46.482" y="59.69" size="1.778" layer="96" rot="R90"/>
-</instance>
-<instance part="CN1" gate="G$1" x="106.68" y="43.18" smashed="yes">
-<attribute name="NAME" x="96.52" y="51.816" size="1.27" layer="95"/>
-<attribute name="VALUE" x="96.52" y="33.02" size="1.27" layer="96"/>
+<instance part="R_1K" gate="G$1" x="106.68" y="45.72" smashed="yes" rot="R90">
+<attribute name="NAME" x="105.1814" y="41.91" size="1.778" layer="95" rot="R90"/>
+<attribute name="VALUE" x="109.982" y="41.91" size="1.778" layer="96" rot="R90"/>
 </instance>
 </instances>
@@
 <segment>
 <pinref part="CONNECTED" gate="G$1" pin="C"/>
-<wire x1="43.18" y1="45.72" x2="43.18" y2="35.56" width="0.1524" layer="91"/>
-<label x="45.72" y="35.56" size="1.778" layer="95"/>
-</segment>
-<segment>
-<pinref part="CN1" gate="G$1" pin="GND"/>
-<wire x1="116.84" y1="38.1" x2="132.08" y2="38.1" width="0.1524" layer="91"/>
-<label x="121.92" y="33.02" size="1.778" layer="95"/>
+<wire x1="53.34" y1="58.42" x2="53.34" y2="48.26" width="0.1524" layer="91"/>
+<label x="60.96" y="50.8" size="1.778" layer="95"/>
 </segment>
 </net>
 <net name="VCC" class="0">
 <segment>
+<pinref part="FRONT_PANEL_INTERFACE" gate="A" pin="2"/>
+<wire x1="0" y1="76.2" x2="17.78" y2="76.2" width="0.1524" layer="91"/>
+<label x="10.16" y="78.74" size="1.778" layer="95" rot="R180"/>
+</segment>
+<segment>
 <pinref part="X1" gate="G$1" pin="VBUS"/>
 <wire x1="86.36" y1="86.36" x2="86.36" y2="101.6" width="0.1524" layer="91"/>
 <label x="78.74" y="91.44" size="1.778" layer="95"/>
+</segment>
+<segment>
+<pinref part="R_1K" gate="G$1" pin="2"/>
+<wire x1="106.68" y1="50.8" x2="106.68" y2="63.5" width="0.1524" layer="91"/>
+<label x="99.06" y="58.42" size="1.778" layer="95"/>
+</segment>
+</net>
+<net name="VCC_1K" class="0">
+<segment>
+<pinref part="FRONT_PANEL_INTERFACE" gate="A" pin="3"/>
+<wire x1="0" y1="78.74" x2="17.78" y2="78.74" width="0.1524" layer="91"/>
+<label x="12.7" y="78.74" size="1.778" layer="95"/>
 </segment>
 <segment>
@@
 </segment>
 <segment>
-<pinref part="R_1K" gate="G$1" pin="2"/>
-<wire x1="43.18" y1="68.58" x2="43.18" y2="76.2" width="0.1524" layer="91"/>
-<label x="45.72" y="73.66" size="1.778" layer="95"/>
+<pinref part="R_1K" gate="G$1" pin="1"/>
+<wire x1="106.68" y1="40.64" x2="106.68" y2="27.94" width="0.1524" layer="91"/>
+<label x="111.76" y="33.02" size="1.778" layer="95"/>
 </segment>
 <segment>
-<pinref part="FRONT_PANEL_INTERFACE" gate="A" pin="6"/>
-<wire x1="0" y1="86.36" x2="15.24" y2="86.36" width="0.1524" layer="91"/>
-<label x="7.62" y="91.44" size="1.778" layer="95"/>
-</segment>
-<segment>
-<pinref part="CN1" gate="G$1" pin="VBUS"/>
-<wire x1="116.84" y1="48.26" x2="129.54" y2="48.26" width="0.1524" layer="91"/>
-<label x="119.38" y="50.8" size="1.778" layer="95"/>
+<pinref part="CONNECTED" gate="G$1" pin="A"/>
+<wire x1="53.34" y1="66.04" x2="53.34" y2="76.2" width="0.1524" layer="91"/>
+<label x="58.42" y="71.12" size="1.778" layer="95"/>
 </segment>
 </net>
-<net name="N$1" class="0">
-<segment>
-<pinref part="R_1K" gate="G$1" pin="1"/>
-<pinref part="CONNECTED" gate="G$1" pin="A"/>
-<wire x1="43.18" y1="58.42" x2="43.18" y2="53.34" width="0.1524" layer="91"/>
-</segment>
-</net>
-<net name="DPLUS" class="0">
-<segment>
-<pinref part="CN1" gate="G$1" pin="D-"/>
-<wire x1="116.84" y1="45.72" x2="129.54" y2="45.72" width="0.1524" layer="91"/>
-<label x="124.46" y="45.72" size="1.778" layer="95"/>
-</segment>
-<segment>
-<pinref part="X1" gate="G$1" pin="D+"/>
-<wire x1="88.9" y1="86.36" x2="88.9" y2="93.98" width="0.1524" layer="91"/>
-<label x="88.9" y="96.52" size="1.778" layer="95" rot="R90"/>
-</segment>
-</net>
-<net name="DMINUS" class="0">
-<segment>
-<pinref part="CN1" gate="G$1" pin="D+"/>
-<wire x1="116.84" y1="43.18" x2="124.46" y2="43.18" width="0.1524" layer="91"/>
-<label x="121.92" y="40.64" size="1.778" layer="95"/>
-</segment>
-<segment>
-<pinref part="X1" gate="G$1" pin="D-"/>
-<wire x1="91.44" y1="86.36" x2="91.44" y2="99.06" width="0.1524" layer="91"/>
-<label x="96.52" y="96.52" size="1.778" layer="95" rot="R90"/>
-</segment>
-</net>
