File: 2023/UpTo11.2023/FrontPanel/bu/UpTo11.FrontPanel.brd (EAGLE design)
At the start: 88 x 78 mm, 16 parts

Commit message: BNSK Booster v 2
Parts:
- moved CONNECTED 61.9 mm to (12.0, 36.0)
- moved R3 3.85 mm to (82.0, 32.2)
- moved DIAL_LED 3.69 mm to (72.0, 32.4)
- moved BOOSTER_ON_LED 0.59 mm to (72.0, 63.0)

Commit message: UpTo11 2023 update
Parts:
- moved SWITCH_OUT 28.6 mm to (58.0, 61.0)
- moved CONNECTED 19.7 mm to (22.0, 19.0)
- moved SWITCH_IN 11.4 mm to (31.3, 58.5)
- moved POT_OUT_(MIDDLE) 3.75 mm to (17.9, 30.1)
- moved R1 3.61 mm to (71.0, 19.0)
- moved POT_IN_(RIGHT) 3.25 mm to (6.71, 30.0)
- moved POT_GND_(LEFT) 3.21 mm to (28.6, 30.2)
Other:
- outline, holes or cut-outs redrawn
