File: 2023/USB Multiplicator 2023/USB Multiplicator 2023.brd (EAGLE design)
At the start: 88 x 78 mm, 10 parts, among them X1 USB-A

Commit message: Fix usb female minus/plus
Connections:
- net USB_DMINUS: now also USB_OUT_WITH_DATA_1.D-; no longer USB_OUT_WITH_DATA_1.D+
- net USB_DPLUS: now also USB_OUT_WITH_DATA_1.D+; no longer USB_OUT_WITH_DATA_1.D-
Routing:
- net GND: track 275.6 -> 0.00 mm
- net VCC: track 225.6 -> 0.00 mm
- net USB_DPLUS: track 80.1 -> 0.00 mm
- net USB_DMINUS: track 75.2 -> 0.00 mm
- net N$5: track 4.05 -> 0.00 mm
Changed lines of the file:
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@@
 <wire x1="8.37043125" y1="12.08465625" x2="2" y2="18.402225" width="0.1524" layer="21" curve="-90"/>
 <rectangle x1="54.95798125" y1="0.15875" x2="55.78601875" y2="0.22225" layer="21"/>
+<rectangle x1="54.95798125" y1="0.22225" x2="55.78601875" y2="0.28575" layer="21"/>
 <rectangle x1="54.95798125" y1="0.28575" x2="55.78601875" y2="0.34925" layer="21"/>
 <rectangle x1="54.95798125" y1="0.34925" x2="55.78601875" y2="0.41275" layer="21"/>
+<rectangle x1="54.95798125" y1="0.41275" x2="55.78601875" y2="0.47625" layer="21"/>
+<rectangle x1="54.95798125" y1="0.47625" x2="55.78601875" y2="0.53975" layer="21"/>
 <rectangle x1="56.164428125" y1="41.867653125" x2="56.992465625" y2="41.931153125" layer="21"/>
 <rectangle x1="56.164428125" y1="41.931153125" x2="56.992465625" y2="41.994653125" layer="21"/>
@@
 <contactref element="USB_OUT_5" pad="GND"/>
 <contactref element="USB_OUT_6" pad="GND"/>
-<wire x1="8.5" y1="17.5" x2="40.5" y2="17.5" width="0.254" layer="1"/>
-<wire x1="8.5" y1="23" x2="8.5" y2="17.5" width="0.254" layer="1"/>
-<wire x1="40.5" y1="17.5" x2="40.5" y2="17.3" width="0.254" layer="1"/>
-<wire x1="8.5" y1="23" x2="8.2" y2="23.4" width="0.254" layer="1"/>
-<wire x1="7" y1="60.5" x2="8" y2="59.5" width="0.254" layer="1"/>
-<wire x1="7" y1="67.5" x2="7" y2="60.5" width="0.254" layer="1"/>
-<wire x1="21" y1="81.5" x2="7" y2="67.5" width="0.254" layer="1"/>
-<wire x1="21" y1="83.5" x2="21" y2="81.5" width="0.254" layer="1"/>
-<wire x1="8" y1="59.5" x2="8.2" y2="59.4" width="0.254" layer="1"/>
-<wire x1="21" y1="83.5" x2="21.4" y2="83.8" width="0.254" layer="1"/>
-<wire x1="7" y1="24.5" x2="8" y2="23.5" width="0.254" layer="1"/>
-<wire x1="7" y1="31.5" x2="7" y2="24.5" width="0.254" layer="1"/>
-<wire x1="8" y1="32.5" x2="7" y2="31.5" width="0.254" layer="1"/>
-<wire x1="8" y1="59" x2="8" y2="32.5" width="0.254" layer="1"/>
-<wire x1="8" y1="23.5" x2="8.2" y2="23.4" width="0.254" layer="1"/>
-<wire x1="8" y1="59" x2="8.2" y2="59.4" width="0.254" layer="1"/>
-<wire x1="44.5" y1="26.5" x2="45.5" y2="25.5" width="0.254" layer="1"/>
-<wire x1="44.5" y1="30.5" x2="44.5" y2="26.5" width="0.254" layer="1"/>
-<wire x1="45" y1="31" x2="44.5" y2="30.5" width="0.254" layer="1"/>
-<wire x1="67" y1="31" x2="45" y2="31" width="0.254" layer="1"/>
-<wire x1="67" y1="22.5" x2="67" y2="31" width="0.254" layer="1"/>
-<wire x1="45.5" y1="25.5" x2="45.848875" y2="25.43760625" width="0.254" layer="1"/>
-<wire x1="67" y1="22.5" x2="67.43" y2="22.5" width="0.254" layer="1"/>
-<wire x1="78" y1="24" x2="83.5" y2="29.5" width="0.254" layer="16"/>
-<wire x1="69" y1="24" x2="78" y2="24" width="0.254" layer="16"/>
-<wire x1="67.5" y1="22.5" x2="69" y2="24" width="0.254" layer="16"/>
-<wire x1="83.5" y1="29.5" x2="83.8" y2="29.6" width="0.254" layer="16"/>
-<wire x1="67.5" y1="22.5" x2="67.43" y2="22.5" width="0.254" layer="16"/>
-<wire x1="85" y1="65.5" x2="84" y2="66.5" width="0.254" layer="1"/>
-<wire x1="85" y1="58.5" x2="85" y2="65.5" width="0.254" layer="1"/>
-<wire x1="84" y1="57.5" x2="85" y2="58.5" width="0.254" layer="1"/>
-<wire x1="84" y1="30" x2="84" y2="57.5" width="0.254" layer="1"/>
-<wire x1="84" y1="66.5" x2="83.8" y2="66.6" width="0.254" layer="1"/>
-<wire x1="84" y1="30" x2="83.8" y2="29.6" width="0.254" layer="1"/>
-<wire x1="64.5" y1="85" x2="63.5" y2="84" width="0.254" layer="16"/>
-<wire x1="71" y1="85" x2="64.5" y2="85" width="0.254" layer="16"/>
-<wire x1="83.5" y1="72.5" x2="71" y2="85" width="0.254" layer="16"/>
-<wire x1="83.5" y1="67" x2="83.5" y2="72.5" width="0.254" layer="16"/>
-<wire x1="63.5" y1="84" x2="63.4" y2="83.8" width="0.254" layer="16"/>
-<wire x1="83.5" y1="67" x2="83.8" y2="66.6" width="0.254" layer="16"/>
-<wire x1="22.5" y1="85" x2="21.5" y2="84" width="0.254" layer="16"/>
-<wire x1="29.5" y1="85" x2="22.5" y2="85" width="0.254" layer="16"/>
-<wire x1="30.5" y1="84" x2="29.5" y2="85" width="0.254" layer="16"/>
-<wire x1="63" y1="84" x2="30.5" y2="84" width="0.254" layer="16"/>
-<wire x1="21.5" y1="84" x2="21.4" y2="83.8" width="0.254" layer="16"/>
-<wire x1="63" y1="84" x2="63.4" y2="83.8" width="0.254" layer="16"/>
+<wire x1="63.4" y1="83.8" x2="83.8" y2="66.6" width="0" layer="19" extent="1-1"/>
+<wire x1="83.8" y1="29.6" x2="83.8" y2="66.6" width="0" layer="19" extent="1-1"/>
+<wire x1="67.43" y1="22.5" x2="83.8" y2="29.6" width="0" layer="19" extent="1-1"/>
+<wire x1="45.848875" y1="25.43760625" x2="67.43" y2="22.5" width="0" layer="19" extent="1-1"/>
+<wire x1="40.5" y1="17.3" x2="45.848875" y2="25.43760625" width="0" layer="19" extent="1-1"/>
+<wire x1="8.2" y1="23.4" x2="40.5" y2="17.3" width="0" layer="19" extent="1-1"/>
+<wire x1="8.2" y1="59.4" x2="8.2" y2="23.4" width="0" layer="19" extent="1-1"/>
+<wire x1="21.4" y1="83.8" x2="8.2" y2="59.4" width="0" layer="19" extent="1-1"/>
 </signal>
 <signal name="VCC">
@@
 <contactref element="USB_OUT_5" pad="VBUS"/>
 <contactref element="USB_OUT_6" pad="VBUS"/>
-<wire x1="9.5" y1="31.5" x2="8.5" y2="30.5" width="0.254" layer="1"/>
-<wire x1="9.5" y1="65" x2="9.5" y2="31.5" width="0.254" layer="1"/>
-<wire x1="8.5" y1="66" x2="9.5" y2="65" width="0.254" layer="1"/>
-<wire x1="8.5" y1="30.5" x2="8.2" y2="30.4" width="0.254" layer="1"/>
-<wire x1="8.5" y1="66" x2="8.2" y2="66.4" width="0.254" layer="1"/>
-<wire x1="11" y1="66.5" x2="28" y2="83.5" width="0.254" layer="16"/>
-<wire x1="8.5" y1="66.5" x2="11" y2="66.5" width="0.254" layer="16"/>
-<wire x1="28" y1="83.5" x2="28.4" y2="83.8" width="0.254" layer="16"/>
-<wire x1="8.5" y1="66.5" x2="8.2" y2="66.4" width="0.254" layer="16"/>
-<wire x1="70.5" y1="73" x2="83.5" y2="60" width="0.254" layer="1"/>
-<wire x1="70.5" y1="83.5" x2="70.5" y2="73" width="0.254" layer="1"/>
-<wire x1="83.5" y1="60" x2="83.8" y2="59.6" width="0.254" layer="1"/>
-<wire x1="70.5" y1="83.5" x2="70.4" y2="83.8" width="0.254" layer="1"/>
-<wire x1="47.5" y1="28" x2="46.5" y2="29" width="0.254" layer="1"/>
-<wire x1="47.5" y1="17.3" x2="47.5" y2="21" width="0.254" layer="1"/>
-<wire x1="47.5" y1="21" x2="47.5" y2="28" width="0.254" layer="1"/>
-<wire x1="46.5" y1="29" x2="46.048875" y2="29.43760625" width="0.254" layer="1"/>
-<wire x1="69.97" y1="22.5" x2="82.5" y2="22.5" width="0.254" layer="1"/>
-<wire x1="82.5" y1="22.5" x2="83.5" y2="22.5" width="0.254" layer="1"/>
-<wire x1="83.5" y1="22.5" x2="83.8" y2="22.6" width="0.254" layer="1"/>
-<wire x1="69.5" y1="21" x2="47.5" y2="21" width="0.254" layer="1"/>
-<wire x1="69.5" y1="22.5" x2="69.5" y2="21" width="0.254" layer="1"/>
-<wire x1="69.5" y1="22.5" x2="69.97" y2="22.5" width="0.254" layer="1"/>
-<wire x1="82.5" y1="58.5" x2="83.5" y2="59.5" width="0.254" layer="1"/>
-<wire x1="82.5" y1="22.5" x2="82.5" y2="58.5" width="0.254" layer="1"/>
-<wire x1="83.5" y1="59.5" x2="83.8" y2="59.6" width="0.254" layer="1"/>
-<wire x1="29.5" y1="82.5" x2="28.5" y2="83.5" width="0.254" layer="16"/>
-<wire x1="69" y1="82.5" x2="29.5" y2="82.5" width="0.254" layer="16"/>
-<wire x1="70" y1="83.5" x2="69" y2="82.5" width="0.254" layer="16"/>
-<wire x1="28.5" y1="83.5" x2="28.4" y2="83.8" width="0.254" layer="16"/>
-<wire x1="70" y1="83.5" x2="70.4" y2="83.8" width="0.254" layer="16"/>
+<wire x1="83.8" y1="59.6" x2="70.4" y2="83.8" width="0" layer="19" extent="1-1"/>
+<wire x1="83.8" y1="22.6" x2="83.8" y2="59.6" width="0" layer="19" extent="1-1"/>
+<wire x1="69.97" y1="22.5" x2="83.8" y2="22.6" width="0" layer="19" extent="1-1"/>
+<wire x1="47.5" y1="17.3" x2="69.97" y2="22.5" width="0" layer="19" extent="1-1"/>
+<wire x1="46.048875" y1="29.43760625" x2="47.5" y2="17.3" width="0" layer="19" extent="1-1"/>
+<wire x1="8.2" y1="30.4" x2="46.048875" y2="29.43760625" width="0" layer="19" extent="1-1"/>
+<wire x1="8.2" y1="66.4" x2="8.2" y2="30.4" width="0" layer="19" extent="1-1"/>
+<wire x1="28.4" y1="83.8" x2="8.2" y2="66.4" width="0" layer="19" extent="1-1"/>
 </signal>
 <signal name="N$5">
 <contactref element="LED_PWR" pad="C"/>
 <contactref element="R_1K" pad="2"/>
-<wire x1="43" y1="29" x2="43" y2="25.5" width="0.254" layer="1"/>
-<wire x1="43" y1="25.5" x2="43.004875" y2="25.43760625" width="0.254" layer="1"/>
-<wire x1="43" y1="29" x2="43.204875" y2="29.43760625" width="0.254" layer="1"/>
+<wire x1="43.004875" y1="25.43760625" x2="43.204875" y2="29.43760625" width="0" layer="19" extent="1-1"/>
 </signal>
 <signal name="USB_DPLUS">
 <contactref element="X1" pad="3"/>
-<contactref element="USB_OUT_WITH_DATA_1" pad="D-"/>
-<wire x1="22.5" y1="38" x2="43" y2="17.5" width="0.254" layer="1"/>
-<wire x1="22.5" y1="84" x2="22.5" y2="38" width="0.254" layer="1"/>
-<wire x1="23.5" y1="85" x2="22.5" y2="84" width="0.254" layer="1"/>
-<wire x1="25.5" y1="85" x2="23.5" y2="85" width="0.254" layer="1"/>
-<wire x1="25.5" y1="84" x2="25.5" y2="85" width="0.254" layer="1"/>
-<wire x1="43" y1="17.5" x2="43" y2="17.3" width="0.254" layer="1"/>
-<wire x1="25.5" y1="84" x2="25.9" y2="83.8" width="0.254" layer="1"/>
+<contactref element="USB_OUT_WITH_DATA_1" pad="D+"/>
+<wire x1="43" y1="17.3" x2="23.9" y2="83.8" width="0" layer="19" extent="1-1"/>
 </signal>
 <signal name="USB_DMINUS">
 <contactref element="X1" pad="2"/>
-<contactref element="USB_OUT_WITH_DATA_1" pad="D+"/>
-<wire x1="43" y1="19.5" x2="45" y2="17.5" width="0.254" layer="1"/>
-<wire x1="43" y1="23" x2="43" y2="19.5" width="0.254" layer="1"/>
-<wire x1="24" y1="42" x2="43" y2="23" width="0.254" layer="1"/>
-<wire x1="24" y1="83.5" x2="24" y2="42" width="0.254" layer="1"/>
-<wire x1="45" y1="17.5" x2="45" y2="17.3" width="0.254" layer="1"/>
-<wire x1="24" y1="83.5" x2="23.9" y2="83.8" width="0.254" layer="1"/>
+<contactref element="USB_OUT_WITH_DATA_1" pad="D-"/>
+<wire x1="45" y1="17.3" x2="25.9" y2="83.8" width="0" layer="19" extent="1-1"/>
 </signal>
 </signals>

Commit message: USB Multiplicator update v2
Routing:
- net GND: track 0.00 -> 251.7 mm
- net VCC: track 0.00 -> 226.5 mm
- net USB_DMINUS: track 0.00 -> 74.5 mm
- net USB_DPLUS: track 0.00 -> 74.4 mm
- net N$5: track 0.00 -> 4.11 mm
Other:
- outline, holes or cut-outs redrawn
- board text added: "PCBv3 - 2023.10"
- board text added: "USB Multiplicator www.FredericTorres.com"
- board text removed: "PCBv3 - 2019.12"
- board text removed: "USB Multiplicator MadeInTheUSB.net"
