File: 2023/USB Multiplicator 2023/bu/USB Multiplicator 2023.brd (EAGLE design)
At the start: 88 x 78 mm, 10 parts, among them X1 USB-A

Commit message: Fix usb female minus/plus
Connections:
- net USB_DMINUS: now also USB_OUT_WITH_DATA_1.D-; no longer USB_OUT_WITH_DATA_1.D+
- net USB_DPLUS: now also USB_OUT_WITH_DATA_1.D+; no longer USB_OUT_WITH_DATA_1.D-
Changed lines of the file:
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@@
 <signal name="USB_DPLUS">
 <contactref element="X1" pad="3"/>
-<contactref element="USB_OUT_WITH_DATA_1" pad="D-"/>
-<wire x1="43" y1="17.3" x2="25.9" y2="83.8" width="0" layer="19" extent="1-1"/>
+<contactref element="USB_OUT_WITH_DATA_1" pad="D+"/>
+<wire x1="43" y1="17.3" x2="23.9" y2="83.8" width="0" layer="19" extent="1-1"/>
 </signal>
 <signal name="USB_DMINUS">
 <contactref element="X1" pad="2"/>
-<contactref element="USB_OUT_WITH_DATA_1" pad="D+"/>
-<wire x1="45" y1="17.3" x2="23.9" y2="83.8" width="0" layer="19" extent="1-1"/>
+<contactref element="USB_OUT_WITH_DATA_1" pad="D-"/>
+<wire x1="45" y1="17.3" x2="25.9" y2="83.8" width="0" layer="19" extent="1-1"/>
 </signal>
 </signals>
