File: 2023/USB Multiplicator 2025/USB Multiplicator 2025.sch (EAGLE design)
At the start: 11 parts, among them X1 USB-A

Commit message: Update...
Connections:
- net USB_DMINUS renamed N$1
- net USB_DPLUS renamed N$2
Other:
- moved on the sheet: X1
Changed lines of the file:
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@@
 </plain>
 <instances>
-<instance part="X1" gate="G$1" x="182.88" y="99.06" smashed="yes" rot="R180">
-<attribute name="NAME" x="193.04" y="90.424" size="1.27" layer="95" rot="R180"/>
-<attribute name="VALUE" x="193.04" y="106.68" size="1.27" layer="96" rot="R180"/>
+<instance part="X1" gate="G$1" x="185.42" y="99.06" smashed="yes" rot="R180">
+<attribute name="NAME" x="195.58" y="90.424" size="1.27" layer="95" rot="R180"/>
+<attribute name="VALUE" x="195.58" y="106.68" size="1.27" layer="96" rot="R180"/>
 </instance>
 <instance part="GND1" gate="1" x="165.1" y="111.76" smashed="yes" rot="R180">
@@
 <attribute name="VALUE" x="-32.385" y="117.348" size="1.778" layer="96" rot="R90"/>
 </instance>
-<instance part="USB_OUT_WITH_DATA_1" gate="G$1" x="55.88" y="104.14" smashed="yes"/>
-<instance part="GND2" gate="1" x="35.56" y="106.68" smashed="yes" rot="R270">
-<attribute name="VALUE" x="33.02" y="109.22" size="1.778" layer="96" rot="R270"/>
+<instance part="USB_OUT_WITH_DATA_1" gate="G$1" x="170.18" y="129.54" smashed="yes"/>
+<instance part="GND2" gate="1" x="149.86" y="132.08" smashed="yes" rot="R270">
+<attribute name="VALUE" x="147.32" y="134.62" size="1.778" layer="96" rot="R270"/>
 </instance>
 <instance part="USB_OUT_2" gate="G$1" x="66.04" y="78.74" smashed="yes"/>
@@
 <segment>
 <pinref part="X1" gate="G$1" pin="GND"/>
-<wire x1="172.72" y1="101.6" x2="165.1" y2="101.6" width="0.1524" layer="91"/>
+<wire x1="175.26" y1="101.6" x2="165.1" y2="101.6" width="0.1524" layer="91"/>
 <pinref part="GND1" gate="1" pin="GND"/>
 <wire x1="165.1" y1="101.6" x2="165.1" y2="109.22" width="0.1524" layer="91"/>
@@
 <pinref part="USB_OUT_WITH_DATA_1" gate="G$1" pin="GND"/>
 <pinref part="GND2" gate="1" pin="GND"/>
-<wire x1="53.34" y1="106.68" x2="38.1" y2="106.68" width="0.1524" layer="91"/>
+<wire x1="167.64" y1="132.08" x2="152.4" y2="132.08" width="0.1524" layer="91"/>
 </segment>
 <segment>
@@
 <segment>
 <pinref part="USB_OUT_WITH_DATA_1" gate="G$1" pin="VBUS"/>
-<wire x1="53.34" y1="109.22" x2="30.48" y2="109.22" width="0.1524" layer="91"/>
-<label x="35.56" y="109.22" size="1.778" layer="95"/>
+<wire x1="167.64" y1="134.62" x2="144.78" y2="134.62" width="0.1524" layer="91"/>
+<label x="149.86" y="134.62" size="1.778" layer="95"/>
 </segment>
 <segment>
@@
 <segment>
 <pinref part="X1" gate="G$1" pin="VBUS"/>
-<wire x1="172.72" y1="93.98" x2="165.1" y2="91.44" width="0.1524" layer="91"/>
+<wire x1="175.26" y1="93.98" x2="165.1" y2="91.44" width="0.1524" layer="91"/>
 <label x="160.02" y="88.9" size="1.778" layer="95"/>
 </segment>
@@
 <wire x1="149.86" y1="55.88" x2="167.64" y2="55.88" width="0.1524" layer="91"/>
 <label x="154.94" y="53.34" size="1.778" layer="95"/>
-</segment>
-</net>
-<net name="USB_DPLUS" class="0">
-<segment>
-<pinref part="X1" gate="G$1" pin="D+"/>
-<wire x1="172.72" y1="96.52" x2="152.4" y2="96.52" width="0.1524" layer="91"/>
-<label x="142.24" y="93.98" size="1.778" layer="95"/>
-</segment>
-<segment>
-<pinref part="USB_OUT_WITH_DATA_1" gate="G$1" pin="D+"/>
-<wire x1="53.34" y1="114.3" x2="25.4" y2="114.3" width="0.1524" layer="91"/>
-<label x="27.94" y="116.84" size="1.778" layer="95"/>
-</segment>
-</net>
-<net name="USB_DMINUS" class="0">
-<segment>
-<pinref part="X1" gate="G$1" pin="D-"/>
-<wire x1="172.72" y1="99.06" x2="152.4" y2="99.06" width="0.1524" layer="91"/>
-<label x="142.24" y="101.6" size="1.778" layer="95"/>
-</segment>
-<segment>
-<pinref part="USB_OUT_WITH_DATA_1" gate="G$1" pin="D-"/>
-<wire x1="53.34" y1="111.76" x2="17.78" y2="111.76" width="0.1524" layer="91"/>
-<label x="20.32" y="111.76" size="1.778" layer="95"/>
 </segment>
 </net>
@@
 </segment>
 </net>
+<net name="N$1" class="0">
+<segment>
+<pinref part="X1" gate="G$1" pin="D-"/>
+<wire x1="175.26" y1="99.06" x2="142.24" y2="99.06" width="0.1524" layer="91"/>
+<wire x1="142.24" y1="99.06" x2="142.24" y2="137.16" width="0.1524" layer="91"/>
+<pinref part="USB_OUT_WITH_DATA_1" gate="G$1" pin="D-"/>
+<wire x1="142.24" y1="137.16" x2="167.64" y2="137.16" width="0.1524" layer="91"/>
+</segment>
+</net>
+<net name="N$2" class="0">
+<segment>
+<pinref part="X1" gate="G$1" pin="D+"/>
+<wire x1="175.26" y1="96.52" x2="137.16" y2="96.52" width="0.1524" layer="91"/>
+<wire x1="137.16" y1="96.52" x2="137.16" y2="139.7" width="0.1524" layer="91"/>
+<pinref part="USB_OUT_WITH_DATA_1" gate="G$1" pin="D+"/>
+<wire x1="137.16" y1="139.7" x2="167.64" y2="139.7" width="0.1524" layer="91"/>
+</segment>
+</net>

Commit message: Update...
Parts:
- added H1, H2, H3, H4: MOUNT-PAD-ROUND3.3, holes:MOUNT-PAD-ROUND3.3
- added JP1: (no value), pinhead:PINHD-1X4
Connections:
- net GND: now also JP1.4
- net VCC: now also JP1.1
Changed lines of the file:
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@@
 <part name="RN1" library="resistor-sip" deviceset="4610X" device=""/>
 <part name="GND9" library="supply1" deviceset="GND" device=""/>
+<part name="JP1" library="pinhead" library_urn="urn:adsk.eagle:library:325" deviceset="PINHD-1X4" device="" package3d_urn="urn:adsk.eagle:package:22407/2"/>
+<part name="GND5" library="supply1" deviceset="GND" device=""/>
+<part name="H1" library="holes" library_urn="urn:adsk.eagle:library:237" deviceset="MOUNT-PAD-ROUND" device="3.3" package3d_urn="urn:adsk.eagle:package:14283/1"/>
+<part name="H2" library="holes" library_urn="urn:adsk.eagle:library:237" deviceset="MOUNT-PAD-ROUND" device="3.3" package3d_urn="urn:adsk.eagle:package:14283/1"/>
+<part name="H3" library="holes" library_urn="urn:adsk.eagle:library:237" deviceset="MOUNT-PAD-ROUND" device="3.3" package3d_urn="urn:adsk.eagle:package:14283/1"/>
+<part name="H4" library="holes" library_urn="urn:adsk.eagle:library:237" deviceset="MOUNT-PAD-ROUND" device="3.3" package3d_urn="urn:adsk.eagle:package:14283/1"/>
 </parts>
 <sheets>
@@
 <attribute name="VALUE" x="-17.78" y="127" size="1.778" layer="96"/>
 </instance>
+<instance part="JP1" gate="A" x="73.66" y="144.78" smashed="yes">
+<attribute name="NAME" x="67.31" y="153.035" size="1.778" layer="95"/>
+<attribute name="VALUE" x="67.31" y="137.16" size="1.778" layer="96"/>
+</instance>
+<instance part="GND5" gate="1" x="48.26" y="142.24" smashed="yes" rot="R270">
+<attribute name="VALUE" x="48.26" y="139.7" size="1.778" layer="96" rot="R270"/>
+</instance>
+<instance part="H1" gate="G$1" x="88.9" y="162.56" smashed="yes">
+<attribute name="NAME" x="91.694" y="163.1442" size="1.778" layer="95"/>
+<attribute name="VALUE" x="91.694" y="160.0962" size="1.778" layer="96"/>
+</instance>
+<instance part="H2" gate="G$1" x="127" y="162.56" smashed="yes">
+<attribute name="NAME" x="129.794" y="163.1442" size="1.778" layer="95"/>
+<attribute name="VALUE" x="129.794" y="160.0962" size="1.778" layer="96"/>
+</instance>
+<instance part="H3" gate="G$1" x="88.9" y="154.94" smashed="yes">
+<attribute name="NAME" x="91.694" y="155.5242" size="1.778" layer="95"/>
+<attribute name="VALUE" x="91.694" y="152.4762" size="1.778" layer="96"/>
+</instance>
+<instance part="H4" gate="G$1" x="124.46" y="154.94" smashed="yes">
+<attribute name="NAME" x="127.254" y="155.5242" size="1.778" layer="95"/>
+<attribute name="VALUE" x="127.254" y="152.4762" size="1.778" layer="96"/>
+</instance>
 </instances>
 <busses>
@@
 <wire x1="-15.24" y1="134.62" x2="-15.24" y2="132.08" width="0.1524" layer="91"/>
 </segment>
+<segment>
+<pinref part="JP1" gate="A" pin="4"/>
+<pinref part="GND5" gate="1" pin="GND"/>
+<wire x1="71.12" y1="142.24" x2="50.8" y2="142.24" width="0.1524" layer="91"/>
+</segment>
 </net>
 <net name="VCC" class="0">
@@
 <wire x1="149.86" y1="55.88" x2="167.64" y2="55.88" width="0.1524" layer="91"/>
 <label x="154.94" y="53.34" size="1.778" layer="95"/>
+</segment>
+<segment>
+<pinref part="JP1" gate="A" pin="1"/>
+<wire x1="71.12" y1="149.86" x2="30.48" y2="149.86" width="0.1524" layer="91"/>
+<label x="38.1" y="147.32" size="1.778" layer="95"/>
 </segment>
 </net>
@@
 </schematic>
 </drawing>
+<compatibility>
+<note version="8.2" severity="warning">
+Since Version 8.2, EAGLE supports online libraries. The ids
+of those online libraries will not be understood (or retained)
+with this version.
+</note>
+<note version="8.3" severity="warning">
+Since Version 8.3, EAGLE supports URNs for individual library
+assets (packages, symbols, and devices). The URNs of those assets
+will not be understood (or retained) with this version.
+</note>
+<note version="8.3" severity="warning">
+Since Version 8.3, EAGLE supports the association of 3D packages
+with devices in libraries, schematics, and board files. Those 3D
+packages will not be understood (or retained) with this version.
+</note>
+</compatibility>
 </eagle>
