File: 2023/USB Multiplicator 2025/bu/USB Multiplicator 2025.brd (EAGLE design)
At the start: 88 x 61 mm, 11 parts, among them X1 USB-A

Commit message: Update...
Parts:
- added H1, H2, H3, H4: MOUNT-PAD-ROUND3.3, holes:3,3-PAD
- added JP1: (no value), pinhead:1X04
- moved USB_OUT_1 2.00 mm to (82.5, 39.0)
- moved USB_OUT_2 2.00 mm to (9.50, 26.0)
Connections:
- net GND: now also JP1.4
- net VCC: now also JP1.1
Other:
- board text added: "VCC 5V"
Changed lines of the file:
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@@
 <text x="43.926875" y="25.93760625" size="1.016" layer="25">+</text>
 <text x="47.58824375" y="24.0302125" size="1.27" layer="25" align="center">POWER</text>
-<text x="70.1" y="17.1" size="2.1844" layer="25" rot="R180" align="center">USB Multiplicator</text>
+<text x="65.1" y="17.1" size="2.1844" layer="25" rot="R180" align="center">USB Multiplicator</text>
 <rectangle x1="54.95798125" y1="0.28575" x2="55.78601875" y2="0.34925" layer="21"/>
 <rectangle x1="54.95798125" y1="0.34925" x2="55.78601875" y2="0.41275" layer="21"/>
@@
 <text x="79.926875" y="46.93760625" size="1.016" layer="25">+</text>
 <text x="29" y="42.7" size="1.016" layer="25">GND</text>
-<text x="13" y="26.7" size="1.016" layer="25">GND</text>
-<text x="76" y="33.7" size="1.016" layer="25">GND</text>
+<text x="13" y="28.7" size="1.016" layer="25">GND</text>
+<text x="76" y="35.7" size="1.016" layer="25">GND</text>
 <text x="41" y="61.7" size="1.016" layer="25">GND</text>
 <wire x1="2" y1="68" x2="2" y2="17" width="0" layer="20"/>
@@
 <wire x1="90" y1="17" x2="85" y2="12" width="0.1524" layer="20" curve="-90"/>
 <wire x1="85" y1="12" x2="84" y2="12" width="0.1524" layer="20"/>
+<text x="72.5" y="67.7" size="1.016" layer="25" rot="R270">GND</text>
+<text x="64.5" y="67.7" size="1.016" layer="25" rot="R270">VCC 5V</text>
 </plain>
 <attributes>
@@
 <attribute name="NAME" x="36.1" y="63.2" size="1.27" layer="25"/>
 </element>
-<element name="USB_OUT_2" library="STUNTAZ" package="USB-FEMALE-A-PTH" value="USB" x="9.5" y="24" smashed="yes" rot="R90">
-<attribute name="NAME" x="11.6" y="26.1" size="1.27" layer="25" rot="R90"/>
+<element name="USB_OUT_2" library="STUNTAZ" package="USB-FEMALE-A-PTH" value="USB" x="9.5" y="26" smashed="yes" rot="R90">
+<attribute name="NAME" x="11.6" y="28.1" size="1.27" layer="25" rot="R90"/>
 </element>
-<element name="USB_OUT_1" library="STUNTAZ" package="USB-FEMALE-A-PTH" value="USB" x="82.5" y="37" smashed="yes" rot="R270">
-<attribute name="NAME" x="80.4" y="34.9" size="1.27" layer="25" rot="R270"/>
+<element name="USB_OUT_1" library="STUNTAZ" package="USB-FEMALE-A-PTH" value="USB" x="82.5" y="39" smashed="yes" rot="R270">
+<attribute name="NAME" x="80.4" y="36.9" size="1.27" layer="25" rot="R270"/>
 </element>
 <element name="S2" library="adafruit" package="EG1218" value="" x="12" y="55" smashed="yes">
@@
 <attribute name="VALUE" x="25.23" y="59.92" size="1.27" layer="27" ratio="10" rot="R90"/>
 </element>
+<element name="JP1" library="pinhead" library_urn="urn:adsk.eagle:library:325" package="1X04" package3d_urn="urn:adsk.eagle:package:22407/2" value="" x="69" y="70" smashed="yes">
+<attribute name="POPULARITY" value="91" x="69" y="70" size="1.778" layer="27" display="off"/>
+<attribute name="VALUE" x="63.92" y="66.825" size="1.27" layer="27"/>
+</element>
+<element name="H1" library="holes" library_urn="urn:adsk.eagle:library:237" package="3,3-PAD" package3d_urn="urn:adsk.eagle:package:14283/1" value="MOUNT-PAD-ROUND3.3" x="8" y="67" smashed="yes">
+<attribute name="POPULARITY" value="1" x="8" y="67" size="1.778" layer="27" display="off"/>
+</element>
+<element name="H2" library="holes" library_urn="urn:adsk.eagle:library:237" package="3,3-PAD" package3d_urn="urn:adsk.eagle:package:14283/1" value="MOUNT-PAD-ROUND3.3" x="8" y="18" smashed="yes">
+<attribute name="POPULARITY" value="1" x="8" y="18" size="1.778" layer="27" display="off"/>
+</element>
+<element name="H3" library="holes" library_urn="urn:adsk.eagle:library:237" package="3,3-PAD" package3d_urn="urn:adsk.eagle:package:14283/1" value="MOUNT-PAD-ROUND3.3" x="84" y="67" smashed="yes">
+<attribute name="POPULARITY" value="1" x="84" y="67" size="1.778" layer="27" display="off"/>
+</element>
+<element name="H4" library="holes" library_urn="urn:adsk.eagle:library:237" package="3,3-PAD" package3d_urn="urn:adsk.eagle:package:14283/1" value="MOUNT-PAD-ROUND3.3" x="84" y="18" smashed="yes">
+<attribute name="POPULARITY" value="1" x="84" y="18" size="1.778" layer="27" display="off"/>
+</element>
 </elements>
 <signals>
@@
 <contactref element="USB_OUT_1" pad="GND"/>
 <contactref element="RN1" pad="1"/>
-<wire x1="65.43" y1="24.5" x2="83.8" y2="33.6" width="0" layer="19" extent="1-1"/>
-<wire x1="40.5" y1="17.3" x2="65.43" y2="24.5" width="0" layer="19" extent="1-1"/>
-<wire x1="27" y1="43.54" x2="40.5" y2="17.3" width="0" layer="19" extent="1-1"/>
-<wire x1="8.2" y1="27.4" x2="27" y2="43.54" width="0" layer="19" extent="1-1"/>
-<wire x1="43.4" y1="66.8" x2="27" y2="43.54" width="0" layer="19" extent="1-1"/>
+<contactref element="JP1" pad="4"/>
+<wire x1="43.4" y1="66.8" x2="72.81" y2="70" width="0" layer="19" extent="1-1"/>
+<wire x1="27" y1="43.54" x2="43.4" y2="66.8" width="0" layer="19" extent="1-1"/>
+<wire x1="8.2" y1="29.4" x2="27" y2="43.54" width="0" layer="19" extent="1-1"/>
+<wire x1="40.5" y1="17.3" x2="27" y2="43.54" width="0" layer="19" extent="1-1"/>
+<wire x1="65.43" y1="24.5" x2="40.5" y2="17.3" width="0" layer="19" extent="1-1"/>
+<wire x1="83.8" y1="35.6" x2="65.43" y2="24.5" width="0" layer="19" extent="1-1"/>
 </signal>
 <signal name="VCC">
@@
 <contactref element="X1" pad="1"/>
 <contactref element="S1" pad="P"/>
+<contactref element="JP1" pad="1"/>
 <wire x1="50.4" y1="66.8" x2="80" y2="55" width="0" layer="19" extent="1-1"/>
 <wire x1="67.97" y1="24.5" x2="80" y2="55" width="0" layer="19" extent="1-1"/>
-<wire x1="46.204875" y1="26.43760625" x2="67.97" y2="24.5" width="0" layer="19" extent="1-1"/>
-<wire x1="47.5" y1="17.3" x2="46.204875" y2="26.43760625" width="0" layer="19" extent="1-1"/>
+<wire x1="47.5" y1="17.3" x2="67.97" y2="24.5" width="0" layer="19" extent="1-1"/>
+<wire x1="46.204875" y1="26.43760625" x2="47.5" y2="17.3" width="0" layer="19" extent="1-1"/>
 <wire x1="12" y1="55" x2="50.4" y2="66.8" width="0" layer="19" extent="1-1"/>
+<wire x1="65.19" y1="70" x2="12" y2="55" width="0" layer="19" extent="1-1"/>
 </signal>
 <signal name="VCC_USB_2">
@@
 <contactref element="USB_OUT_2" pad="VBUS"/>
 <contactref element="LED_PWR2" pad="A"/>
-<wire x1="8.2" y1="34.4" x2="9.46" y2="55" width="0" layer="19" extent="1-1"/>
-<wire x1="6.578" y1="48" x2="8.2" y2="34.4" width="0" layer="19" extent="1-1"/>
+<wire x1="6.578" y1="48" x2="9.46" y2="55" width="0" layer="19" extent="1-1"/>
+<wire x1="8.2" y1="36.4" x2="6.578" y2="48" width="0" layer="19" extent="1-1"/>
 </signal>
 <signal name="VCC_USB_3">
@@
 <contactref element="S1" pad="O"/>
 <wire x1="82.578" y1="48" x2="82.54" y2="55" width="0" layer="19" extent="1-1"/>
-<wire x1="83.8" y1="26.6" x2="82.578" y2="48" width="0" layer="19" extent="1-1"/>
+<wire x1="83.8" y1="28.6" x2="82.578" y2="48" width="0" layer="19" extent="1-1"/>
 </signal>
 <signal name="R1">
@@
 which will not be processed correctly with this version.
 </note>
+<note version="8.2" severity="warning">
+Since Version 8.2, EAGLE supports online libraries. The ids
+of those online libraries will not be understood (or retained)
+with this version.
+</note>
+<note version="8.3" severity="warning">
+Since Version 8.3, EAGLE supports URNs for individual library
+assets (packages, symbols, and devices). The URNs of those assets
+will not be understood (or retained) with this version.
+</note>
+<note version="8.3" severity="warning">
+Since Version 8.3, EAGLE supports the association of 3D packages
+with devices in libraries, schematics, and board files. Those 3D
+packages will not be understood (or retained) with this version.
+</note>
 </compatibility>
