File: NUSBIO BOARD/Nusbio1.0.WaveShare.I2C.LCD/bu.v1/Nusbio1.0.WaveShare.I2C.LCD.sch (EAGLE design)
At the start: 17 parts

Commit message: Update...
Parts:
- removed BUTTON_1_GPIO_1: (no value), switch-omron:10-XX
- removed LED_2_GPIO_2: (no value), adafruit:LEDSMT1206
Connections:
- removed net BUTTON_2_R: BUTTON_1_GPIO_1.P1, RN1.6
- removed net LED_2_R: LED_2_GPIO_2.C, RN1.3
- net DCD_G3: now also U$1.4; no longer LED_2_GPIO_2.A
- net DTR_G2: now also U$1.3; no longer BUTTON_1_GPIO_1.S
Changed lines of the file:
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@@
 <part name="BUTTON_1_GPIO_0" library="switch-omron" library_urn="urn:adsk.eagle:library:377" deviceset="10-XX" device="" package3d_urn="urn:adsk.eagle:package:27496/1"/>
 <part name="LED_1_GPIO_1" library="adafruit" deviceset="LED" device="SMT1206"/>
-<part name="BUTTON_1_GPIO_1" library="switch-omron" library_urn="urn:adsk.eagle:library:377" deviceset="10-XX" device="" package3d_urn="urn:adsk.eagle:package:27496/1"/>
-<part name="LED_2_GPIO_2" library="adafruit" deviceset="LED" device="SMT1206"/>
 </parts>
 <sheets>
@@
 <attribute name="VALUE" x="207.645" y="57.912" size="1.778" layer="96" rot="R270"/>
 </instance>
-<instance part="BUTTON_1_GPIO_1" gate="1" x="279.4" y="30.48" smashed="yes">
-<attribute name="NAME" x="273.05" y="27.94" size="1.778" layer="95" rot="R90"/>
-<attribute name="VALUE" x="275.59" y="33.655" size="1.778" layer="96" rot="R90"/>
-</instance>
-<instance part="LED_2_GPIO_2" gate="G$1" x="213.36" y="-2.54" smashed="yes" rot="R180">
-<attribute name="NAME" x="209.804" y="2.032" size="1.778" layer="95" rot="R270"/>
-<attribute name="VALUE" x="207.645" y="2.032" size="1.778" layer="96" rot="R270"/>
-</instance>
 </instances>
 <busses>
@@
 </segment>
 <segment>
-<pinref part="LED_2_GPIO_2" gate="G$1" pin="A"/>
-<wire x1="213.36" y1="-5.08" x2="213.36" y2="-22.86" width="0.1524" layer="91"/>
-<wire x1="213.36" y1="-22.86" x2="215.9" y2="-22.86" width="0.1524" layer="91"/>
-<label x="220.98" y="-15.24" size="1.778" layer="95"/>
+<pinref part="U$1" gate="G$1" pin="4"/>
+<wire x1="134.62" y1="76.2" x2="114.3" y2="76.2" width="0.1524" layer="91"/>
+<label x="114.3" y="76.2" size="1.778" layer="95"/>
 </segment>
 </net>
@@
 </segment>
 <segment>
-<pinref part="BUTTON_1_GPIO_1" gate="1" pin="S"/>
-<wire x1="279.4" y1="35.56" x2="279.4" y2="60.96" width="0.1524" layer="91"/>
-<wire x1="279.4" y1="60.96" x2="281.94" y2="60.96" width="0.1524" layer="91"/>
-<label x="279.4" y="63.5" size="1.778" layer="95"/>
+<pinref part="U$1" gate="G$1" pin="3"/>
+<wire x1="134.62" y1="78.74" x2="114.3" y2="78.74" width="0.1524" layer="91"/>
+<label x="114.3" y="78.74" size="1.778" layer="95"/>
 </segment>
 </net>
@@
 <pinref part="RN1" gate="G$1" pin="5"/>
 <wire x1="162.56" y1="76.2" x2="162.56" y2="60.96" width="0.1524" layer="91"/>
+<wire x1="162.56" y1="60.96" x2="165.1" y2="60.96" width="0.1524" layer="91"/>
 <label x="160.02" y="68.58" size="1.778" layer="95" rot="R270"/>
 </segment>
@@
 </segment>
 </net>
-<net name="BUTTON_2_R" class="0">
-<segment>
-<pinref part="RN1" gate="G$1" pin="6"/>
-<wire x1="165.1" y1="76.2" x2="165.1" y2="43.18" width="0.1524" layer="91"/>
-<label x="165.1" y="40.64" size="1.778" layer="95" rot="R90"/>
-</segment>
-<segment>
-<pinref part="BUTTON_1_GPIO_1" gate="1" pin="P1"/>
-<wire x1="281.94" y1="25.4" x2="281.94" y2="0" width="0.1524" layer="91"/>
-<label x="284.48" y="2.54" size="1.778" layer="95"/>
-</segment>
-</net>
-<net name="LED_2_R" class="0">
-<segment>
-<pinref part="RN1" gate="G$1" pin="3"/>
-<wire x1="157.48" y1="76.2" x2="157.48" y2="60.96" width="0.1524" layer="91"/>
-<label x="157.48" y="60.96" size="1.778" layer="95" rot="R90"/>
-</segment>
-<segment>
-<pinref part="LED_2_GPIO_2" gate="G$1" pin="C"/>
-<wire x1="213.36" y1="2.54" x2="213.36" y2="20.32" width="0.1524" layer="91"/>
-<label x="215.9" y="12.7" size="1.778" layer="95"/>
-</segment>
-</net>
